File: _saved_SmallKat v2.sch (KiCad schematic (older format))
At the start: 59 parts, among them IC1 TPS562201DDCR, J1 Conn_01x06_Male, J10 Conn_01x03_Male, J11 Conn_01x03_Male, J12 Conn_01x03_Male, J13 Conn_01x03_Male, J14 Conn_01x03_Male, J15 Conn_01x03_Male, J16 Conn_01x03_Male, J17 Conn_01x03_Male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

Commit message: Updated to use BECs and added silkscreen
Parts:
- gave numbers to parts that had none: 8
Connections:
- net +6V is gone; now on net +BATT: C19.1, C21.1, C22.1, IC1.3 (VIN), R11.1
Changed lines of the file:
@@
-$EndComp
-$Comp
-L power:+6V #PWR0136
-U 1 1 5C5A30D0
-P 4400 5500
-F 0 "#PWR0136" H 4400 5350 50  0001 C CNN
-F 1 "+6V" V 4415 5628 50  0000 L CNN
-F 2 "" H 4400 5500 50  0001 C CNN
-F 3 "" H 4400 5500 50  0001 C CNN
-	1    4400 5500
-	0    1    1    0
 $EndComp
 $Comp
@@
 BATTMONITOR
 $Comp
-L power:+6V #PWR0174
-U 1 1 5C5F62BF
-P 2400 5800
-F 0 "#PWR0174" H 2400 5650 50  0001 C CNN
-F 1 "+6V" V 2415 5928 50  0000 L CNN
-F 2 "" H 2400 5800 50  0001 C CNN
-F 3 "" H 2400 5800 50  0001 C CNN
-	1    2400 5800
-	0    -1   -1   0
-$EndComp
-Connection ~ 2400 5800
-$Comp
-L Connector:Conn_01x02_Male J?
+L Connector:Conn_01x02_Male J22
 U 1 1 5C6FA8A3
 P 4550 6500
-F 0 "J?" V 4610 6540 50  0000 L CNN
+F 0 "J22" V 4610 6540 50  0000 L CNN
 F 1 "Conn_01x02_Male" V 4701 6540 50  0000 L CNN
 F 2 "Connector_PinHeader_2.54mm:PinHeader_1x02_P2.54mm_Vertical" H 4550 6500 50  0001 C CNN
@@
 $EndComp
 $Comp
-L power:GND #PWR?
+L power:GND #PWR0109
 U 1 1 5C6FA8B0
 P 4550 6700
-F 0 "#PWR?" H 4550 6450 50  0001 C CNN
+F 0 "#PWR0109" H 4550 6450 50  0001 C CNN
 F 1 "GND" H 4555 6527 50  0000 C CNN
 F 2 "" H 4550 6700 50  0001 C CNN
@@
 $EndComp
 $Comp
-L Connector:Conn_01x02_Male J?
+L Connector:Conn_01x02_Male J24
 U 1 1 5C6FAF58
 P 4900 6500
-F 0 "J?" V 4960 6540 50  0000 L CNN
+F 0 "J24" V 4960 6540 50  0000 L CNN
 F 1 "Conn_01x02_Male" V 5051 6540 50  0000 L CNN
 F 2 "Connector_PinHeader_2.54mm:PinHeader_1x02_P2.54mm_Vertical" H 4900 6500 50  0001 C CNN
@@
 $EndComp
 $Comp
-L power:GND #PWR?
+L power:GND #PWR0110
 U 1 1 5C6FAF65
 P 4900 6700
-F 0 "#PWR?" H 4900 6450 50  0001 C CNN
+F 0 "#PWR0110" H 4900 6450 50  0001 C CNN
 F 1 "GND" H 4905 6527 50  0000 C CNN
 F 2 "" H 4900 6700 50  0001 C CNN
@@
 $EndComp
 $Comp
-L Connector:Conn_01x02_Male J?
+L Connector:Conn_01x02_Male J27
 U 1 1 5C6FB610
 P 5250 6500
-F 0 "J?" V 5310 6540 50  0000 L CNN
+F 0 "J27" V 5310 6540 50  0000 L CNN
 F 1 "Conn_01x02_Male" V 5401 6540 50  0000 L CNN
 F 2 "Connector_PinHeader_2.54mm:PinHeader_1x02_P2.54mm_Vertical" H 5250 6500 50  0001 C CNN
@@
 $EndComp
 $Comp
-L power:GND #PWR?
+L power:GND #PWR0122
 U 1 1 5C6FB61D
 P 5250 6700
-F 0 "#PWR?" H 5250 6450 50  0001 C CNN
+F 0 "#PWR0122" H 5250 6450 50  0001 C CNN
 F 1 "GND" H 5255 6527 50  0000 C CNN
 F 2 "" H 5250 6700 50  0001 C CNN
@@
 $EndComp
 $Comp
-L Connector:Conn_01x02_Male J?
+L Connector:Conn_01x02_Male J29
 U 1 1 5C6FBCD7
 P 5600 6500
-F 0 "J?" V 5660 6540 50  0000 L CNN
+F 0 "J29" V 5660 6540 50  0000 L CNN
 F 1 "Conn_01x02_Male" V 5751 6540 50  0000 L CNN
 F 2 "Connector_PinHeader_2.54mm:PinHeader_1x02_P2.54mm_Vertical" H 5600 6500 50  0001 C CNN
@@
 $EndComp
 $Comp
-L power:GND #PWR?
+L power:GND #PWR0123
 U 1 1 5C6FBCE4
 P 5600 6700
-F 0 "#PWR?" H 5600 6450 50  0001 C CNN
+F 0 "#PWR0123" H 5600 6450 50  0001 C CNN
 F 1 "GND" H 5605 6527 50  0000 C CNN
 F 2 "" H 5600 6700 50  0001 C CNN
@@
 +6V_IN4
 $Comp
-L Connector:Conn_01x02_Male J?
+L Connector:Conn_01x02_Male J23
 U 1 1 5C6FD52B
 P 4550 7100
-F 0 "J?" V 4610 7140 50  0000 L CNN
+F 0 "J23" V 4610 7140 50  0000 L CNN
 F 1 "Conn_01x02_Male" V 4701 7140 50  0000 L CNN
 F 2 "Connector_PinHeader_2.54mm:PinHeader_1x02_P2.54mm_Vertical" H 4550 7100 50  0001 C CNN
@@
 $EndComp
 $Comp
-L power:+BATT #PWR?
+L power:+BATT #PWR0124
 U 1 1 5C6FD532
 P 4450 7300
-F 0 "#PWR?" H 4450 7150 50  0001 C CNN
+F 0 "#PWR0124" H 4450 7150 50  0001 C CNN
 F 1 "+BATT" H 4465 7473 50  0000 C CNN
 F 2 "" H 4450 7300 50  0001 C CNN
@@
 $EndComp
 $Comp
-L power:GND #PWR?
+L power:GND #PWR0125
 U 1 1 5C6FD538
 P 4550 7300
-F 0 "#PWR?" H 4550 7050 50  0001 C CNN
+F 0 "#PWR0125" H 4550 7050 50  0001 C CNN
 F 1 "GND" H 4555 7127 50  0000 C CNN
 F 2 "" H 4550 7300 50  0001 C CNN
@@
 $EndComp
 $Comp
-L Connector:Conn_01x02_Male J?
+L Connector:Conn_01x02_Male J25
 U 1 1 5C6FDBE8
 P 4900 7100
-F 0 "J?" V 4960 7140 50  0000 L CNN
+F 0 "J25" V 4960 7140 50  0000 L CNN
 F 1 "Conn_01x02_Male" V 5051 7140 50  0000 L CNN
 F 2 "Connector_PinHeader_2.54mm:PinHeader_1x02_P2.54mm_Vertical" H 4900 7100 50  0001 C CNN
@@
 $EndComp
 $Comp
-L power:+BATT #PWR?
+L power:+BATT #PWR0126
 U 1 1 5C6FDBEF
 P 4800 7300
-F 0 "#PWR?" H 4800 7150 50  0001 C CNN
+F 0 "#PWR0126" H 4800 7150 50  0001 C CNN
 F 1 "+BATT" H 4815 7473 50  0000 C CNN
 F 2 "" H 4800 7300 50  0001 C CNN
@@
 $EndComp
 $Comp
-L power:GND #PWR?
+L power:GND #PWR0127
 U 1 1 5C6FDBF5
 P 4900 7300
-F 0 "#PWR?" H 4900 7050 50  0001 C CNN
+F 0 "#PWR0127" H 4900 7050 50  0001 C CNN
 F 1 "GND" H 4905 7127 50  0000 C CNN
 F 2 "" H 4900 7300 50  0001 C CNN
@@
 $EndComp
 $Comp
-L Connector:Conn_01x02_Male J?
+L Connector:Conn_01x02_Male J26
 U 1 1 5C6FE2A0
 P 5150 7100
-F 0 "J?" V 5210 7140 50  0000 L CNN
+F 0 "J26" V 5210 7140 50  0000 L CNN
 F 1 "Conn_01x02_Male" V 5301 7140 50  0000 L CNN
 F 2 "Connector_PinHeader_2.54mm:PinHeader_1x02_P2.54mm_Vertical" H 5150 7100 50  0001 C CNN
@@
 $EndComp
 $Comp
-L power:+BATT #PWR?
+L power:+BATT #PWR0128
 U 1 1 5C6FE2A7
 P 5050 7300
-F 0 "#PWR?" H 5050 7150 50  0001 C CNN
+F 0 "#PWR0128" H 5050 7150 50  0001 C CNN
 F 1 "+BATT" H 5065 7473 50  0000 C CNN
 F 2 "" H 5050 7300 50  0001 C CNN
@@
 $EndComp
 $Comp
-L power:GND #PWR?
+L power:GND #PWR0129
 U 1 1 5C6FE2AD
 P 5150 7300
-F 0 "#PWR?" H 5150 7050 50  0001 C CNN
+F 0 "#PWR0129" H 5150 7050 50  0001 C CNN
 F 1 "GND" H 5155 7127 50  0000 C CNN
 F 2 "" H 5150 7300 50  0001 C CNN
@@
 $EndComp
 $Comp
-L Connector:Conn_01x02_Male J?
+L Connector:Conn_01x02_Male J28
 U 1 1 5C6FE959
 P 5400 7100
-F 0 "J?" V 5460 7140 50  0000 L CNN
+F 0 "J28" V 5460 7140 50  0000 L CNN
 F 1 "Conn_01x02_Male" V 5551 7140 50  0000 L CNN
 F 2 "Connector_PinHeader_2.54mm:PinHeader_1x02_P2.54mm_Vertical" H 5400 7100 50  0001 C CNN
@@
 $EndComp
 $Comp
-L power:+BATT #PWR?
+L power:+BATT #PWR0130
 U 1 1 5C6FE960
 P 5300 7300
-F 0 "#PWR?" H 5300 7150 50  0001 C CNN
+F 0 "#PWR0130" H 5300 7150 50  0001 C CNN
 F 1 "+BATT" H 5315 7473 50  0000 C CNN
 F 2 "" H 5300 7300 50  0001 C CNN
@@
 $EndComp
 $Comp
-L power:GND #PWR?
+L power:GND #PWR0131
 U 1 1 5C6FE966
 P 5400 7300
-F 0 "#PWR?" H 5400 7050 50  0001 C CNN
+F 0 "#PWR0131" H 5400 7050 50  0001 C CNN
 F 1 "GND" H 5405 7127 50  0000 C CNN
 F 2 "" H 5400 7300 50  0001 C CNN
@@
 	1    0    0    -1
 $EndComp
+$Comp
+L power:+BATT #PWR0132
+U 1 1 5C700DEA
+P 4400 5500
+F 0 "#PWR0132" H 4400 5350 50  0001 C CNN
+F 1 "+BATT" H 4415 5673 50  0000 C CNN
+F 2 "" H 4400 5500 50  0001 C CNN
+F 3 "" H 4400 5500 50  0001 C CNN
+	1    4400 5500
+	0    1    1    0
+$EndComp
+$Comp
+L power:+BATT #PWR0133
+U 1 1 5C700F1C
+P 2400 5800
+F 0 "#PWR0133" H 2400 5650 50  0001 C CNN
+F 1 "+BATT" H 2415 5973 50  0000 C CNN
+F 2 "" H 2400 5800 50  0001 C CNN
+F 3 "" H 2400 5800 50  0001 C CNN
+	1    2400 5800
+	0    -1   -1   0
+$EndComp
+Connection ~ 2400 5800
 $EndSCHEMATC
