File: SmallKat v2.sch (KiCad schematic (older format))
At the start: 59 parts, among them IC1 TPS562201DDCR, J1 Conn_01x06_Male, J10 Conn_01x03_Male, J11 Conn_01x03_Male, J12 Conn_01x03_Male, J13 Conn_01x03_Male, J14 Conn_01x03_Male, J15 Conn_01x03_Male, J16 Conn_01x03_Male, J17 Conn_01x03_Male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

Commit message: Updated to use nucleo l432kc
Parts:
- removed U1: ESP32-DEVKITC-32D, ESP32-DEVKITC-32D:MODULE_ESP32-DEVKITC-32D, symbol ESP32-DEVKITC-32D:ESP32-DEVKITC-32D
- added J30: Conn_01x15_Female, Connector_PinSocket_2.54mm:PinSocket_1x15_P2.54mm_Vertical, symbol Connector:Conn_01x15_Female
- added J31: Conn_01x15_Female, Connector_PinHeader_2.54mm:PinHeader_1x15_P2.54mm_Vertical, symbol Connector:Conn_01x15_Female
- J29: renamed from J?; footprint Connector_PinHeader_2.54mm:PinHeader_1x02_P2.54mm_Vertical -> Connector_PinSocket_2.54mm:PinSocket_1x15_P2.54mm_Vertical
- R12: value 39.5k -> 61.63k
- gave numbers to parts that had none: 7
Connections:
- net labels added: +5V
- net labels removed: +6V
- no-connect marks 0 -> 2

Commit message: init
Parts:
- removed C18, C20: 22uF, Capacitor_SMD:C_0805_2012Metric, symbol Device:C
- removed C19: 10Uf, Capacitor_SMD:C_0805_2012Metric, symbol Device:C
- removed C21, C24: 10uF, Capacitor_SMD:C_0805_2012Metric, symbol Device:C
- removed C22, C23, C25: 0.1uF, Capacitor_SMD:C_0402_1005Metric, symbol Device:C
- removed C26, C27: 10pF, Capacitor_SMD:C_0402_1005Metric, symbol Device:C
- removed D1: DIODE, Diode_SMD:D_0805_2012Metric, symbol pspice:DIODE
- removed F1, F2, F3, F4: Fuse, Fuse:Fuse_0805_2012Metric, symbol Device:Fuse
- removed IC1: TPS562201DDCR, TPS562201DDCR:SOT95P280X110-6N, symbol TPS562201DDCR:TPS562201DDCR
- removed J1, J2, J3, J4: Conn_01x06_Male, Connector_PinHeader_1.27mm:PinHeader_1x06_P1.27mm_Vertical, symbol Connector:Conn_01x06_Male
- removed J10, J11, J12, J13, J14, J15, J16, J17, J18, J19, J20, J5, J6, J7, J8, J9: Conn_01x03_Male, Connector_PinHeader_2.54mm:PinHeader_1x03_P2.54mm_Vertical, symbol Connector:Conn_01x03_Male
- removed J21, J22, J23, J24, J25, J26, J27, J28: Conn_01x02_Male, Connector_PinHeader_2.54mm:PinHeader_1x02_P2.54mm_Vertical, symbol Connector:Conn_01x02_Male
- removed J29: Conn_01x02_Male, Connector_PinSocket_2.54mm:PinSocket_1x15_P2.54mm_Vertical, symbol Connector:Conn_01x02_Male
- removed J30: Conn_01x15_Female, Connector_PinSocket_2.54mm:PinSocket_1x15_P2.54mm_Vertical, symbol Connector:Conn_01x15_Female
- removed J31: Conn_01x15_Female, Connector_PinHeader_2.54mm:PinHeader_1x15_P2.54mm_Vertical, symbol Connector:Conn_01x15_Female
- removed L2: 4.7uH, Inductor_SMD:L_0805_2012Metric_Pad1.15x1.40mm_HandSolder, symbol Device:L
- removed R10, R11, R13, R14, R15, R18, R19: 10K, Resistor_SMD:R_0402_1005Metric, symbol Device:R
- removed R12: 61.63k, Resistor_SMD:R_0402_1005Metric, symbol Device:R
- removed R20: 6.2k, Resistor_SMD:R_0402_1005Metric, symbol Device:R
- removed U3: PCA9685BS, Package_DFN_QFN:QFN-28-1EP_6x6mm_P0.65mm_EP4.25x4.25mm, symbol Driver_LED:PCA9685BS
- removed U4: BNO055, Package_LGA:LGA-28_5.2x3.8mm_P0.5mm, symbol Sensor_Motion:BNO055
- removed Y1: 32.768kHz, Crystal:Crystal_SMD_3215-2Pin_3.2x1.5mm, symbol Device:Crystal
Connections:
- no-connect marks 2 -> 0
