File: SmallKat v2.sch (KiCad schematic (older format))
At the start: 0 parts

Commit message: Routing done
Changed lines of the file:
@@
 $Descr A3 16535 11693
 encoding utf-8
-Sheet 1 14
+Sheet 1 12
 Title ""
 Date ""
@@
 F1 "MainBoard.sch" 50
 $EndSheet
-$Sheet
-S 8000 4400 850  1650
-U 5DAA9E7A
-F0 "ControllerBoard" 50
-F1 "ControllerBoard.sch" 50
-$EndSheet
 $EndSCHEMATC
