File: ControllerBoard.sch (KiCad schematic (older format))
At the start: 28 parts, among them J18 Conn_01x02_Male, U10 MIC5365-3.3YC5, U5 MCP73831-2-OT, U9 WIICHUCK

Commit message: Routing done
Parts:
- TP17, TP18, TP19: footprint TestPoint:TestPoint_Pad_D2.5mm -> TestPoint:TestPoint_Pad_D1.5mm
Changed lines of the file:
@@
 F 0 "TP17" H 3958 2968 50  0000 L CNN
 F 1 "TestPoint" H 3958 2877 50  0000 L CNN
-F 2 "TestPoint:TestPoint_Pad_D2.5mm" H 4100 2850 50  0001 C CNN
+F 2 "TestPoint:TestPoint_Pad_D1.5mm" H 4100 2850 50  0001 C CNN
 F 3 "~" H 4100 2850 50  0001 C CNN
 	1    3900 2850
@@
 F 0 "TP18" H 4458 2968 50  0000 L CNN
 F 1 "TestPoint" H 4458 2877 50  0000 L CNN
-F 2 "TestPoint:TestPoint_Pad_D2.5mm" H 4600 2850 50  0001 C CNN
+F 2 "TestPoint:TestPoint_Pad_D1.5mm" H 4600 2850 50  0001 C CNN
 F 3 "~" H 4600 2850 50  0001 C CNN
 	1    4400 2850
@@
 F 0 "TP19" H 1458 918 50  0000 L CNN
 F 1 "TestPoint" H 1458 827 50  0000 L CNN
-F 2 "TestPoint:TestPoint_Pad_D2.5mm" H 1600 800 50  0001 C CNN
+F 2 "TestPoint:TestPoint_Pad_D1.5mm" H 1600 800 50  0001 C CNN
 F 3 "~" H 1600 800 50  0001 C CNN
 	1    1400 800
