File: Servos.sch (KiCad schematic (older format))
At the start: 88 parts, among them IC4 MAX34409ETE+, IC5 MAX34409ETE+, IC6 MAX34409ETE+, IC7 MAX34409ETE+, J1 Conn_01x03_Male, J10 Conn_01x03_Male, J11 Conn_01x03_Male, J12 Conn_01x03_Male, J13 Conn_01x03_Male, J14 Conn_01x03_Male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

Commit message: Changed FP lib to local copy, updated board
Parts:
- F1, F2, F3, F4: footprint 01550900M:0154.250DR -> 0154:0154.250DR
- IC4, IC5, IC6, IC7: symbol MAX34409ETE+:MAX34409ETE+ -> SmallKat-v2-rescue:MAX34409ETE+-MAX34409ETE+
Changed lines of the file:
@@
 EESchema Schematic File Version 4
-LIBS:SmallKat v2-cache
 EELAYER 30 0
 EELAYER END
@@
 F 0 "F1" H 1510 7296 50  0000 L CNN
 F 1 "Fuse" H 1510 7205 50  0000 L CNN
-F 2 "01550900M:0154.250DR" V 1380 7250 50  0001 C CNN
+F 2 "0154:0154.250DR" V 1380 7250 50  0001 C CNN
 F 3 "~" H 1450 7250 50  0001 C CNN
 	1    1450 7250
@@
 	1450 6950 1450 7100
 $Comp
-L MAX34409ETE+:MAX34409ETE+ IC4
+L SmallKat-v2-rescue:MAX34409ETE+-MAX34409ETE+ IC4
 U 1 1 5DD76E19
 P 1050 5250
@@
 F 0 "F2" H 2610 7296 50  0000 L CNN
 F 1 "Fuse" H 2610 7205 50  0000 L CNN
-F 2 "01550900M:0154.250DR" V 2480 7250 50  0001 C CNN
+F 2 "0154:0154.250DR" V 2480 7250 50  0001 C CNN
 F 3 "~" H 2550 7250 50  0001 C CNN
 	1    2550 7250
@@
 F 0 "F3" H 3660 7296 50  0000 L CNN
 F 1 "Fuse" H 3660 7205 50  0000 L CNN
-F 2 "01550900M:0154.250DR" V 3530 7250 50  0001 C CNN
+F 2 "0154:0154.250DR" V 3530 7250 50  0001 C CNN
 F 3 "~" H 3600 7250 50  0001 C CNN
 	1    3600 7250
@@
 F 0 "F4" H 4710 7296 50  0000 L CNN
 F 1 "Fuse" H 4710 7205 50  0000 L CNN
-F 2 "01550900M:0154.250DR" V 4580 7250 50  0001 C CNN
+F 2 "0154:0154.250DR" V 4580 7250 50  0001 C CNN
 F 3 "~" H 4650 7250 50  0001 C CNN
 	1    4650 7250
@@
 NoConn ~ 2250 5450
 $Comp
-L MAX34409ETE+:MAX34409ETE+ IC5
+L SmallKat-v2-rescue:MAX34409ETE+-MAX34409ETE+ IC5
 U 1 1 5DDCC7B0
 P 3450 5250
@@
 NoConn ~ 4650 5450
 $Comp
-L MAX34409ETE+:MAX34409ETE+ IC6
+L SmallKat-v2-rescue:MAX34409ETE+-MAX34409ETE+ IC6
 U 1 1 5DDD3560
 P 5800 5200
@@
 NoConn ~ 7000 5400
 $Comp
-L MAX34409ETE+:MAX34409ETE+ IC7
+L SmallKat-v2-rescue:MAX34409ETE+-MAX34409ETE+ IC7
 U 1 1 5DDD943E
 P 8200 5150
