File: Servos.sch (KiCad schematic (older format))
At the start: 88 parts, among them IC4 MAX34409ETE+, IC5 MAX34409ETE+, IC6 MAX34409ETE+, IC7 MAX34409ETE+, J1 Conn_01x03_Male, J10 Conn_01x03_Male, J11 Conn_01x03_Male, J12 Conn_01x03_Male, J13 Conn_01x03_Male, J14 Conn_01x03_Male, J15 Conn_01x03_Male, J16 Conn_01x03_Male, J17 Conn_01x03_Male, J2 Conn_01x03_Male, J3 Conn_01x03_Male, J4 Conn_01x03_Male, J5 Conn_01x03_Male, J6 Conn_01x03_Male, J7 Conn_01x03_Male, J8 Conn_01x03_Male

Commit message: Routing done
Changed lines of the file:
@@
 $Descr A4 11693 8268
 encoding utf-8
-Sheet 10 14
+Sheet 10 12
 Title ""
 Date ""
@@
 $EndComp
 Connection ~ 3700 3800
-$Comp
-L Device:R R76
-U 1 1 5DDCC7FB
-P 3300 5250
-F 0 "R76" V 3093 5250 50  0000 C CNN
-F 1 "100R" V 3184 5250 50  0000 C CNN
-F 2 "Resistor_SMD:R_0402_1005Metric" V 3230 5250 50  0001 C CNN
-F 3 "~" H 3300 5250 50  0001 C CNN
-	1    3300 5250
-	0    1    1    0
-$EndComp
-Text Label 3150 5250 2    50   ~ 0
+Text Label 4250 4350 1    50   ~ 0
 S5
 $Comp
@@
 	1    0    0    -1
 $EndComp
-Text Label 3850 6550 3    50   ~ 0
+Text Label 3150 5250 0    50   ~ 0
 S6
 $Comp
@@
 	0    -1   -1   0
 $EndComp
+Text Label 3850 6550 3    50   ~ 0
+S7
 Text Label 4950 5550 0    50   ~ 0
-S7
-$Comp
-L Device:R R85
-U 1 1 5DDCC810
-P 4250 4500
-F 0 "R85" V 4043 4500 50  0000 C CNN
-F 1 "100R" V 4134 4500 50  0000 C CNN
-F 2 "Resistor_SMD:R_0402_1005Metric" V 4180 4500 50  0001 C CNN
-F 3 "~" H 4250 4500 50  0001 C CNN
-	1    4250 4500
-	-1   0    0    1
-$EndComp
-Text Label 4250 4350 1    50   ~ 0
 S8
 $Comp
@@
 	0    1    1    0
 $EndComp
-Text Label 5500 5200 2    50   ~ 0
+Text Label 7300 5500 0    50   ~ 0
 S9
 $Comp
@@
 	1    0    0    -1
 $EndComp
-Text Label 6200 6500 3    50   ~ 0
+Text Label 6600 4300 1    50   ~ 0
 S10
 $Comp
@@
 	0    -1   -1   0
 $EndComp
-Text Label 7300 5500 0    50   ~ 0
+Text Label 6200 6500 3    50   ~ 0
 S11
 $Comp
@@
 	-1   0    0    1
 $EndComp
-Text Label 6600 4300 1    50   ~ 0
+Text Label 5500 5200 2    50   ~ 0
 S12
 $Comp
@@
 $EndComp
 Text Label 9000 4250 1    50   ~ 0
-S6
+S16
 $Comp
 L power:GND #PWR0294
@@
 Text HLabel 7550 2300 3    50   Input ~ 0
 SERVO16
+$Comp
+L Device:R R85
+U 1 1 5DDCC810
+P 4250 4500
+F 0 "R85" V 4043 4500 50  0000 C CNN
+F 1 "100R" V 4134 4500 50  0000 C CNN
+F 2 "Resistor_SMD:R_0402_1005Metric" V 4180 4500 50  0001 C CNN
+F 3 "~" H 4250 4500 50  0001 C CNN
+	1    4250 4500
+	-1   0    0    1
+$EndComp
+$Comp
+L Device:R R76
+U 1 1 5DDCC7FB
+P 3300 5250
+F 0 "R76" V 3093 5250 50  0000 C CNN
+F 1 "100R" V 3184 5250 50  0000 C CNN
+F 2 "Resistor_SMD:R_0402_1005Metric" V 3230 5250 50  0001 C CNN
+F 3 "~" H 3300 5250 50  0001 C CNN
+	1    3300 5250
+	0    1    1    0
+$EndComp
 $EndSCHEMATC

Commit message: order
Parts:
- IC4, IC5, IC6, IC7: symbol MAX34409ETE+:MAX34409ETE+ -> SmallKat-v2-rescue:MAX34409ETE+-MAX34409ETE+
Changed lines of the file:
@@
 EESchema Schematic File Version 4
-LIBS:SmallKat v2-cache
 EELAYER 30 0
 EELAYER END
 $Descr A4 11693 8268
 encoding utf-8
-Sheet 10 12
+Sheet 9 12
 Title ""
 Date ""
@@
 	1450 6950 1450 7100
 $Comp
-L MAX34409ETE+:MAX34409ETE+ IC4
+L SmallKat-v2-rescue:MAX34409ETE+-MAX34409ETE+ IC4
 U 1 1 5DD76E19
 P 1050 5250
@@
 NoConn ~ 2250 5450
 $Comp
-L MAX34409ETE+:MAX34409ETE+ IC5
+L SmallKat-v2-rescue:MAX34409ETE+-MAX34409ETE+ IC5
 U 1 1 5DDCC7B0
 P 3450 5250
@@
 NoConn ~ 4650 5450
 $Comp
-L MAX34409ETE+:MAX34409ETE+ IC6
+L SmallKat-v2-rescue:MAX34409ETE+-MAX34409ETE+ IC6
 U 1 1 5DDD3560
 P 5800 5200
@@
 NoConn ~ 7000 5400
 $Comp
-L MAX34409ETE+:MAX34409ETE+ IC7
+L SmallKat-v2-rescue:MAX34409ETE+-MAX34409ETE+ IC7
 U 1 1 5DDD943E
 P 8200 5150

Commit message: Rev
Parts:
- removed C54, C55: 0.1uF, Capacitor_SMD:C_0402_1005Metric, symbol Device:C
- removed IC4, IC5, IC6, IC7: MAX34409ETE+, MAX34409ETE+:QFN65P400X400X80-17N, symbol SmallKat-v2-rescue:MAX34409ETE+-MAX34409ETE+
- removed R101, R102, R103, R106, R107, R108, R109, R111, R112, R113, R114, R59, R60, R64, R65, R67, R68, R71, R72, R76, R77, R81, R82, R84, R85, R89, R90, R93, R94, R95, R96, R98: 100R, Resistor_SMD:R_0402_1005Metric, symbol Device:R
- removed R110, R83, R97: 0R, Resistor_SMD:R_0402_1005Metric, symbol Device:R
- added C37, C42, C43: 0.1uF, Capacitor_SMD:C_0402_1005Metric, symbol Device:C
- added D9: LED, LED_SMD:LED_0603_1608Metric, symbol Device:LED
- added F5: Fuse, 01550900M:0154.250DR, symbol Device:Fuse
- added J18, J20, J22, J23: Conn_01x03_Male, Connector_PinHeader_2.54mm:PinHeader_1x03_P2.54mm_Vertical, symbol Connector:Conn_01x03_Male
- added PS1, PS2, PS3, PS4, PS5: PAC1934T-I_JQ, PAC1934T-I_JQ:QFN65P400X400X55-17N-D, symbol PAC1934T-I_JQ:PAC1934T-I_JQ
- added R128: 20K, Resistor_SMD:R_0402_1005Metric, symbol Device:R
- added R29, R30, R39, R40: 0R, Resistor_SMD:R_0402_1005Metric, symbol Device:R
- added R33, R34, R35, R36: 0.01R, Resistor_SMD:R_0603_1608Metric, symbol Device:R
Connections:
- net labels added: 6V5, S17, S18, S19, S20, SERVO17, SERVO18, SERVO19, SERVO20
- wire segments 44 -> 50
- no-connect marks 8 -> 10
Other:
- moved on the sheet: C52, C53, R66

Commit message: This rev removes the safety micro and instead uses the dji battery
Parts:
- removed C37, C42, C43, C52, C53: 0.1uF, Capacitor_SMD:C_0402_1005Metric, symbol Device:C
- removed D9: LED, LED_SMD:LED_0603_1608Metric, symbol Device:LED
- removed F5: Fuse, 01550900M:0154.250DR, symbol Device:Fuse
- removed J18, J20, J22, J23: Conn_01x03_Male, Connector_PinHeader_2.54mm:PinHeader_1x03_P2.54mm_Vertical, symbol Connector:Conn_01x03_Male
- removed PS1, PS2, PS3, PS4, PS5: PAC1934T-I_JQ, PAC1934T-I_JQ:QFN65P400X400X55-17N-D, symbol PAC1934T-I_JQ:PAC1934T-I_JQ
- removed R100, R104, R105, R61, R62, R69, R70, R74, R75, R79, R80, R87, R88, R91, R92, R99: 0.01R, Resistor_SMD:R_0603_1608Metric, symbol Device:R
- removed R128: 20K, Resistor_SMD:R_0402_1005Metric, symbol Device:R
- removed R29, R30, R39, R40, R66: 0R, Resistor_SMD:R_0402_1005Metric, symbol Device:R
- added R31, R37: 10K, Resistor_SMD:R_0402_1005Metric, symbol Device:R
- added R32, R38: 8.2K, Resistor_SMD:R_0402_1005Metric, symbol Device:R
- R33, R35: value 0.01R -> 10K; footprint Resistor_SMD:R_0603_1608Metric -> Resistor_SMD:R_0402_1005Metric
- R34, R36: value 0.01R -> 8.2K; footprint Resistor_SMD:R_0603_1608Metric -> Resistor_SMD:R_0402_1005Metric
Connections:
- net labels added: MEASURED_FUSE1, MEASURED_FUSE2, MEASURED_FUSE3, MEASURED_FUSE4
- net labels removed: +3.3V, 6V5, S1, S10, S11, S12, S13, S14, S15, S16, S17, S18, S19, S2, S20, S3, S4, S5, S6, S7, S8, S9, SCL, SDA, SERVO17, SERVO18, SERVO19, SERVO20
- wire segments 50 -> 4
- no-connect marks 10 -> 0
Other:
- moved on the sheet: D23, D24, D25, D26, F1, F2, F3, F4, J10, J11, J12, J13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

Commit message: g
Parts:
- renumbered D24 to D10, D25 to D11, D26 to D12, D23 to D9, F1 to F2, F2 to F3, F3 to F4, F4 to F5, J2 to J10, J3 to J11, J4 to J12, J5 to J13, J6 to J14, J7 to J15, J8 to J16, J10 to J17, J11 to J18, J12 to J19, J13 to J20, J14 to J21, J15 to J22, J16 to J23, J17 to J24, J1 to J9, R31 to R24, R32 to R25, R63 to R26, R33 to R27, R34 to R28, R73 to R29, R35 to R30, R36 to R31, R78 to R32, R37 to R33, R38 to R34, R86 to R35
