File: ESP32Module.sch (KiCad schematic (older format))
At the start: 27 parts, among them J20 USB_C_Receptacle, Q3 MMBT3904, Q4 MMBT3904, SW1 SW_SPST, SW2 SW_SPST, U3 ESP32-WROOM-32, U4 CP2102N-A01-GQFN24

Commit message: Use new local FP lib
Parts:
- J20: footprint Connector_USB:USB_C_Receptacle_Amphenol_12401610E4-2A_CircularHoles -> USB_C_Receptacle_Amphenol_12401610E4-2A:USB_C_Receptacle_Amphenol_12401610E4-2A_CircularHoles
Changed lines of the file:
@@
 EESchema Schematic File Version 4
-LIBS:SmallKat v2-cache
 EELAYER 30 0
 EELAYER END
@@
 F 0 "J19" V 4353 8380 50  0000 L CNN
 F 1 "USB_C_Receptacle" V 4262 8380 50  0000 L CNN
-F 2 "Connector_USB:USB_C_Receptacle_Amphenol_12401610E4-2A_CircularHoles" H 4350 7250 50  0001 C CNN
+F 2 "USB_C_Receptacle_Amphenol_12401610E4-2A:USB_C_Receptacle_Amphenol_12401610E4-2A_CircularHoles" H 4350 7250 50  0001 C CNN
 F 3 "https://www.usb.org/sites/default/files/documents/usb_type-c.zip" H 4350 7250 50  0001 C CNN
 	1    4200 7250
