File: ESP32Module.sch (KiCad schematic (older format))
At the start: 32 parts, among them J20 USB_C_Receptacle, Q3 MMBT3904, Q4 MMBT3904, SW1 SW_SPST, SW2 SW_SPST, U2 MIC5365-3.3YC5, U3 ESP32-WROOM-32, U4 CP2102N-A01-GQFN24

Commit message: In progress of charging implimentation
Parts:
- removed C23, C25: 1uF, Capacitor_SMD:C_0402_1005Metric, symbol Device:C
- removed D5: D_TVS, Diode_SMD:D_SOD-523, symbol Device:D_TVS
- removed D6: D_Schottky, Diode_SMD:D_SOD-323, symbol Device:D_Schottky
- removed R22: 10K, Resistor_SMD:R_0402_1005Metric, symbol Device:R
- removed R23: 20K, Resistor_SMD:R_0402_1005Metric, symbol Device:R
- removed U2: MIC5365-3.3YC5, Package_TO_SOT_SMD:SOT-23-5, symbol Regulator_Linear:MIC5365-3.3YC5
- added R4, R5: 10K, Resistor_SMD:R_0402_1005Metric, symbol Device:R
- J20: footprint U263-241N-4BQC11-1:U263241N4BQC111 -> Connector_USB:USB_C_Receptacle_Amphenol_12401610E4-2A_CircularHoles
Connections:
- net labels added: CC1, CC2, VBUS
- net labels removed: +5V
- wire segments 40 -> 35
- no-connect marks 31 -> 29

Commit message: Routing done
Parts:
- TP10, TP11, TP12, TP9: footprint TestPoint:TestPoint_Pad_D2.5mm -> TestPoint:TestPoint_Pad_D1.5mm
Changed lines of the file:
@@
 $Descr A4 11693 8268
 encoding utf-8
-Sheet 6 14
+Sheet 6 12
 Title ""
 Date ""
@@
 F 0 "TP9" H 8958 1068 50  0000 L CNN
 F 1 "TestPoint" H 8958 977 50  0000 L CNN
-F 2 "TestPoint:TestPoint_Pad_D2.5mm" H 9100 950 50  0001 C CNN
+F 2 "TestPoint:TestPoint_Pad_D1.5mm" H 9100 950 50  0001 C CNN
 F 3 "~" H 9100 950 50  0001 C CNN
 	1    8900 950
@@
 F 0 "TP11" H 9508 1068 50  0000 L CNN
 F 1 "TestPoint" H 9508 977 50  0000 L CNN
-F 2 "TestPoint:TestPoint_Pad_D2.5mm" H 9650 950 50  0001 C CNN
+F 2 "TestPoint:TestPoint_Pad_D1.5mm" H 9650 950 50  0001 C CNN
 F 3 "~" H 9650 950 50  0001 C CNN
 	1    9450 950
@@
 F 0 "TP12" H 10058 1068 50  0000 L CNN
 F 1 "TestPoint" H 10058 977 50  0000 L CNN
-F 2 "TestPoint:TestPoint_Pad_D2.5mm" H 10200 950 50  0001 C CNN
+F 2 "TestPoint:TestPoint_Pad_D1.5mm" H 10200 950 50  0001 C CNN
 F 3 "~" H 10200 950 50  0001 C CNN
 	1    10000 950
@@
 F 0 "TP10" H 8958 1418 50  0000 L CNN
 F 1 "TestPoint" H 8958 1327 50  0000 L CNN
-F 2 "TestPoint:TestPoint_Pad_D2.5mm" H 9100 1300 50  0001 C CNN
+F 2 "TestPoint:TestPoint_Pad_D1.5mm" H 9100 1300 50  0001 C CNN
 F 3 "~" H 9100 1300 50  0001 C CNN
 	1    8900 1300

Commit message: Rev
Parts:
- removed Q3, Q4: MMBT3904, Package_TO_SOT_SMD:SOT-23, symbol Transistor_BJT:MMBT3904
- added Q3: MBT3904DW1, Package_TO_SOT_SMD:SOT-363_SC-70-6, symbol Transistor_BJT:MBT3904DW1
- J20: footprint Connector_USB:USB_C_Receptacle_Amphenol_12401610E4-2A_CircularHoles -> C167321:C167321
Changed lines of the file:
@@
-	1    0    0    -1
-$EndComp
-$Comp
-L Transistor_BJT:MMBT3904 Q4
-U 1 1 5DAFB01E
-P 10100 4150
-AR Path="/5DAA9390/5DAAB924/5DAFB01E" Ref="Q4"  Part="1"
-AR Path="/5DAA9E7A/5DB7E2D8/5DAFB01E" Ref="Q6"  Part="1"
-AR Path="/5DB7E2D8/5DAFB01E" Ref="Q4"  Part="1"
-F 0 "Q4" H 10291 4104 50  0000 L CNN
-F 1 "MMBT3904" H 10291 4195 50  0000 L CNN
-F 2 "Package_TO_SOT_SMD:SOT-23" H 10300 4075 50  0001 L CIN
-F 3 "https://www.fairchildsemi.com/datasheets/2N/2N3904.pdf" H 10100 4150 50  0001 L CNN
-	1    10100 4150
-	1    0    0    1
-$EndComp
-$Comp
-L Transistor_BJT:MMBT3904 Q3
-U 1 1 5DAFD0BE
-P 10100 3400
-AR Path="/5DAA9390/5DAAB924/5DAFD0BE" Ref="Q3"  Part="1"
-AR Path="/5DAA9E7A/5DB7E2D8/5DAFD0BE" Ref="Q5"  Part="1"
-AR Path="/5DB7E2D8/5DAFD0BE" Ref="Q3"  Part="1"
-F 0 "Q3" H 10291 3446 50  0000 L CNN
-F 1 "MMBT3904" H 10291 3355 50  0000 L CNN
-F 2 "Package_TO_SOT_SMD:SOT-23" H 10300 3325 50  0001 L CIN
-F 3 "https://www.fairchildsemi.com/datasheets/2N/2N3904.pdf" H 10100 3400 50  0001 L CNN
-	1    10100 3400
 	1    0    0    -1
 $EndComp
@@
 F 0 "J19" V 4353 8380 50  0000 L CNN
 F 1 "USB_C_Receptacle" V 4262 8380 50  0000 L CNN
-F 2 "Connector_USB:USB_C_Receptacle_Amphenol_12401610E4-2A_CircularHoles" H 4350 7250 50  0001 C CNN
+F 2 "C167321:C167321" H 4350 7250 50  0001 C CNN
 F 3 "https://www.usb.org/sites/default/files/documents/usb_type-c.zip" H 4350 7250 50  0001 C CNN
 	1    4200 7250
@@
 	1    0    0    -1
 $EndComp
+$Comp
+L Transistor_BJT:MBT3904DW1 Q3
+U 1 1 5E7A985B
+P 10100 3400
+F 0 "Q3" H 10290 3446 50  0000 L CNN
+F 1 "MBT3904DW1" H 10290 3355 50  0000 L CNN
+F 2 "Package_TO_SOT_SMD:SOT-363_SC-70-6" H 10300 3500 50  0001 C CNN
+F 3 "http://www.onsemi.com/pub_link/Collateral/MBT3904DW1T1-D.PDF" H 10100 3400 50  0001 C CNN
+	1    10100 3400
+	1    0    0    -1
+$EndComp
+$Comp
+L Transistor_BJT:MBT3904DW1 Q3
+U 2 1 5E7AB9F4
+P 10100 4150
+F 0 "Q3" H 10290 4196 50  0000 L CNN
+F 1 "MBT3904DW1" H 10290 4105 50  0000 L CNN
+F 2 "Package_TO_SOT_SMD:SOT-363_SC-70-6" H 10300 4250 50  0001 C CNN
+F 3 "http://www.onsemi.com/pub_link/Collateral/MBT3904DW1T1-D.PDF" H 10100 4150 50  0001 C CNN
+	2    10100 4150
+	1    0    0    -1
+$EndComp

Commit message: This rev removes the safety micro and instead uses the dji battery
Parts:
- removed R24: 470R, Resistor_SMD:R_0402_1005Metric, symbol Device:R
Connections:
- net labels added: IO35, IO36, IO39
- net labels removed: ADC1, CC1, CC2
- no-connect marks 29 -> 27
Changed lines of the file:
@@
 $Descr A4 11693 8268
 encoding utf-8
-Sheet 5 12
+Sheet 5 7
 Title ""
 Date ""
@@
 	1    0    0    -1
 $EndComp
-NoConn ~ 2050 1600
-NoConn ~ 2050 1700
 Wire Wire Line
 	3250 1400 3450 1400
@@
 Wire Wire Line
 	8000 2550 8100 2550
-$Comp
-L Device:R R24
-U 1 1 5DB25907
-P 8250 2550
-AR Path="/5DAA9390/5DAAB924/5DB25907" Ref="R24"  Part="1"
-AR Path="/5DAA9E7A/5DB7E2D8/5DB25907" Ref="R39"  Part="1"
-AR Path="/5DB7E2D8/5DB25907" Ref="R24"  Part="1"
-F 0 "R24" V 8350 2650 50  0000 C CNN
-F 1 "470R" V 8350 2450 50  0000 C CNN
-F 2 "Resistor_SMD:R_0402_1005Metric" V 8180 2550 50  0001 C CNN
-F 3 "~" H 8250 2550 50  0001 C CNN
-	1    8250 2550
-	0    1    1    0
-$EndComp
-Text Label 8400 2550 0    50   ~ 0
+Text Label 8100 2550 0    50   ~ 0
 TXD
 Text Label 8000 2650 0    50   ~ 0
@@
 IO34
 Text HLabel 3250 3700 2    50   Input ~ 0
-ADC1
+IO35
 Text HLabel 3250 2800 2    50   Input ~ 0
 SDA
@@
 NoConn ~ 4900 6650
 NoConn ~ 5100 6650
-Connection ~ 4000 6650
-Connection ~ 3800 6650
-$Comp
-L Connector:USB_C_Receptacle J20
-U 1 1 5DBC0E27
-P 4200 7250
-AR Path="/5DAA9E7A/5DB7E2D8/5DBC0E27" Ref="J20"  Part="1"
-AR Path="/5DAA9390/5DAAB924/5DBC0E27" Ref="J19"  Part="1"
-AR Path="/5DB7E2D8/5DBC0E27" Ref="J19"  Part="1"
-F 0 "J19" V 4353 8380 50  0000 L CNN
-F 1 "USB_C_Receptacle" V 4262 8380 50  0000 L CNN
-F 2 "C167321:C167321" H 4350 7250 50  0001 C CNN
-F 3 "https://www.usb.org/sites/default/files/documents/usb_type-c.zip" H 4350 7250 50  0001 C CNN
-	1    4200 7250
-	0    -1   -1   0
-$EndComp
 NoConn ~ 5200 6650
 NoConn ~ 5400 6650
@@
 Text HLabel 7200 5100 1    50   Input ~ 0
 SCL
-Text HLabel 3400 6650 1    50   Input ~ 0
-CC1
-Text HLabel 3500 6650 1    50   Input ~ 0
-CC2
 $Comp
 L power:+3.3V #PWR0168
@@
 	1    0    0    -1
 $EndComp
+Connection ~ 3800 6650
+Connection ~ 4000 6650
+$Comp
+L Connector:USB_C_Receptacle J20
+U 1 1 5DBC0E27
+P 4200 7250
+AR Path="/5DAA9E7A/5DB7E2D8/5DBC0E27" Ref="J20"  Part="1"
+AR Path="/5DAA9390/5DAAB924/5DBC0E27" Ref="J19"  Part="1"
+AR Path="/5DB7E2D8/5DBC0E27" Ref="J19"  Part="1"
+F 0 "J19" V 4353 8380 50  0000 L CNN
+F 1 "USB_C_Receptacle" V 4262 8380 50  0000 L CNN
+F 2 "C167321:C167321" H 4350 7250 50  0001 C CNN
+F 3 "https://www.usb.org/sites/default/files/documents/usb_type-c.zip" H 4350 7250 50  0001 C CNN
+	1    4200 7250
+	0    -1   -1   0
+$EndComp
+Text HLabel 2050 1600 0    50   Input ~ 0
+IO36
+Text HLabel 2050 1700 0    50   Input ~ 0
+IO39
 $EndSCHEMATC

Commit message: batt connector and all in the right place. has not been ordered, waiting for prev rev to be tested first
Parts:
- J20: symbol Connector:USB_C_Receptacle -> SmallKat-v2-rescue:USB_C_Receptacle-Connector-SmallKat-v2-rescue
Changed lines of the file:
@@
 Connection ~ 4000 6650
 $Comp
-L Connector:USB_C_Receptacle J20
+L SmallKat-v2-rescue:USB_C_Receptacle-Connector-SmallKat-v2-rescue J20
 U 1 1 5DBC0E27
 P 4200 7250
@@
 AR Path="/5DAA9390/5DAAB924/5DBC0E27" Ref="J19"  Part="1"
 AR Path="/5DB7E2D8/5DBC0E27" Ref="J19"  Part="1"
+AR Path="/5DBC0E27" Ref="J19"  Part="1"
 F 0 "J19" V 4353 8380 50  0000 L CNN
 F 1 "USB_C_Receptacle" V 4262 8380 50  0000 L CNN

Commit message: rev, pendingorder
Parts:
- J20: symbol SmallKat-v2-rescue:USB_C_Receptacle-Connector-SmallKat-v2-rescue -> SmallKat-v2-rescue:USB_C_Receptacle-Connector-SmallKat-v2-rescue-SmallKat-v2-rescue-SmallKat-v2-rescue-SmallKat-v2-resc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

Commit message: g
Parts:
- J8: renamed from J20; symbol SmallKat-v2-rescue:USB_C_Receptacle-Connector-SmallKat-v2-rescue-SmallKat-v2-rescue-SmallKat-v2-rescue-SmallKat-v2-rescue -> SmallKat-v2-rescue:USB_C_Receptacle-Connector-SmallKat-v2-rescue-SmallKat-v2-rescue-SmallKat-v2-rescue-SmallKat-v2-rescue-SmallKat-v2-rescue-SmallKat-v2-rescue
- SW1, SW2: footprint Button_Switch_SMD:SW_SPST_CK_KXT3 -> Button_Switch_SMD:SW_SPST_EVQPE1
- renumbered C24 to C17, C26 to C18, C27 to C19, C28 to C20, C29 to C21, C31 to C22, C32 to C23, Q3 to Q1, R21 to R18, R4 to R19, R5 to R20, R25 to R21, R26 to R22, R27 to R23, TP9 to TP5, TP10 to TP6, TP11 to TP7, TP12 to TP8
