File: 6vSwitchMode.sch (KiCad schematic (older format))
At the start: 28 parts, among them IC2 TPS40192DRCT, Q1 BUK9M120-100EX, Q2 BUK9M120-100EX

Commit message: swapped to local FP
Parts:
- IC2: symbol TPS40192DRCT:TPS40192DRCT -> SmallKat-v2-rescue:TPS40192DRCT-TPS40192DRCT
- L2: footprint Inductor_SMD:L_Bourns_SRP1245A -> L_Bourns_SRP1245A:L_Bourns_SRP1245A
Changed lines of the file:
@@
 EESchema Schematic File Version 4
-LIBS:SmallKat v2-cache
 EELAYER 30 0
 EELAYER END
@@
 $EndDescr
 $Comp
-L TPS40192DRCT:TPS40192DRCT IC?
+L SmallKat-v2-rescue:TPS40192DRCT-TPS40192DRCT IC?
 U 1 1 5DAD8199
 P 5100 2900
@@
 F 0 "L2" V 7540 3250 50  0000 C CNN
 F 1 "1uH" V 7449 3250 50  0000 C CNN
-F 2 "Inductor_SMD:L_Bourns_SRP1245A" H 7350 3250 50  0001 C CNN
+F 2 "L_Bourns_SRP1245A:L_Bourns_SRP1245A" H 7350 3250 50  0001 C CNN
 F 3 "~" H 7350 3250 50  0001 C CNN
 	1    7350 3250
