File: 6vSwitchMode.sch (KiCad schematic (older format))
At the start: 28 parts, among them IC2 TPS40192DRCT, Q1 BUK9M120-100EX, Q2 BUK9M120-100EX

Commit message: Routing done
Parts:
- TP6, TP7, TP8: footprint TestPoint:TestPoint_Pad_D2.5mm -> TestPoint:TestPoint_Pad_D1.5mm
Changed lines of the file:
@@
 $Descr A4 11693 8268
 encoding utf-8
-Sheet 5 14
+Sheet 5 12
 Title ""
 Date ""
@@
 F 0 "TP8" H 9608 1568 50  0000 L CNN
 F 1 "TestPoint" H 9608 1477 50  0000 L CNN
-F 2 "TestPoint:TestPoint_Pad_D2.5mm" H 9750 1450 50  0001 C CNN
+F 2 "TestPoint:TestPoint_Pad_D1.5mm" H 9750 1450 50  0001 C CNN
 F 3 "~" H 9750 1450 50  0001 C CNN
 	1    9550 1450
@@
 F 0 "TP7" H 9058 1568 50  0000 L CNN
 F 1 "TestPoint" H 9058 1477 50  0000 L CNN
-F 2 "TestPoint:TestPoint_Pad_D2.5mm" H 9200 1450 50  0001 C CNN
+F 2 "TestPoint:TestPoint_Pad_D1.5mm" H 9200 1450 50  0001 C CNN
 F 3 "~" H 9200 1450 50  0001 C CNN
 	1    9000 1450
@@
 F 0 "TP6" H 8508 1568 50  0000 L CNN
 F 1 "TestPoint" H 8508 1477 50  0000 L CNN
-F 2 "TestPoint:TestPoint_Pad_D2.5mm" H 8650 1450 50  0001 C CNN
+F 2 "TestPoint:TestPoint_Pad_D1.5mm" H 8650 1450 50  0001 C CNN
 F 3 "~" H 8650 1450 50  0001 C CNN
 	1    8450 1450

Commit message: order
Parts:
- removed C10: 1000pF, Capacitor_SMD:C_0402_1005Metric, symbol Device:C
- removed C11: 100pF, Capacitor_SMD:C_0402_1005Metric, symbol Device:C
- removed C22: 1uF, Capacitor_SMD:C_0402_1005Metric, symbol Device:C
- removed IC2: TPS40192DRCT, TPS40192DRCT:SON50P300X300X100-11N, symbol TPS40192DRCT:TPS40192DRCT
- removed R12: 2.18k, Resistor_SMD:R_0402_1005Metric, symbol Device:R
- added C16: 5.6nF, Capacitor_SMD:C_0402_1005Metric, symbol Device:C
- added C18: 1pF, Capacitor_SMD:C_0402_1005Metric, symbol Device:C
- added R20: 18K, Resistor_SMD:R_0402_1005Metric, symbol Device:R
- added R29: 2.74K, Resistor_SMD:R_0402_1005Metric, symbol Device:R
- added R30: 29.4R, Resistor_SMD:R_0402_1005Metric, symbol Device:R
- added U2: LM25145RGYR, LM25145:LM25145RGYR, symbol 2019-12-31_22-15-16:LM25145RGYR
- C12: value 10nF -> 2.2uF
- C13: value 1uF -> 0.1uF
- C14: value 4.7uF -> 6.8nF
- C15: value 470nF -> 0.1uF
- C19: value 100uF -> 330pF; footprint Capacitor_SMD:C_1210_3225Metric -> Capacitor_SMD:C_0402_1005Metric
- C21: value 100uF -> 10uF; footprint Capacitor_SMD:C_1210_3225Metric -> Capacitor_SMD:C_0805_2012Metric
- R13: value 20k -> 2.1R
- R14: value 2.61k -> 10K
- R15: value 4.22k -> 10K
- R16: value 3.9k -> 20K
- R17: value 100k -> 20K
- R18: value 100k -> 634R
- R19: value 100k -> 2.49K
Connections:
- net labels removed: GNDA
- wire segments 50 -> 39
- no-connect marks 0 -> 3
Other:
- moved on the sheet: C10, C11, D4, L2, Q1, Q2, R12, TP4, TP6, TP7

Commit message: Rev
Parts:
- removed C16: 5.6nF, Capacitor_SMD:C_0402_1005Metric, symbol Device:C
- removed C18: 1pF, Capacitor_SMD:C_0402_1005Metric, symbol Device:C
- removed R20: 18K, Resistor_SMD:R_0402_1005Metric, symbol Device:R
- removed R29: 2.74K, Resistor_SMD:R_0402_1005Metric, symbol Device:R
- removed R30: 29.4R, Resistor_SMD:R_0402_1005Metric, symbol Device:R
- removed U2: LM25145RGYR, LM25145:LM25145RGYR, symbol 2019-12-31_22-15-16:LM25145RGYR
- added C10: 1000pF, Capacitor_SMD:C_0402_1005Metric, symbol Device:C
- added C11: 100pF, Capacitor_SMD:C_0402_1005Metric, symbol Device:C
- added C17, C20: 47uF, Capacitor_SMD:C_1206_3216Metric, symbol Device:C
- added C22: 1uF, Capacitor_SMD:C_0402_1005Metric, symbol Device:C
- added IC8: TPS40192DRCT-TPS40192DRCT, Package_SON:VSON-10-1EP_3x3mm_P0.5mm_EP1.2x2mm, symbol SmallKat-v2-rescue:TPS40192DRCT-TPS40192DRCT
- added R12: 2.18k, Resistor_SMD:R_0402_1005Metric, symbol Device:R
- C12: value 2.2uF -> 10nF
- C13: value 0.1uF -> 1uF
- C14: value 6.8nF -> 4.7uF
- C15: value 0.1uF -> 470nF
- C19: value 330pF -> 100uF; footprint Capacitor_SMD:C_0402_1005Metric -> Capacitor_SMD:C_1210_3225Metric
- C21: value 10uF -> 100uF; footprint Capacitor_SMD:C_0805_2012Metric -> Capacitor_SMD:C_1210_3225Metric
- R13: value 2.1R -> 20k
- R14: value 10K -> 2.61k
- R15: value 10K -> 4.22k
- R16: value 20K -> 3.9k
- R17: value 20K -> 100k
- R18: value 634R -> 100k
- R19: value 2.49K -> 100k
- R20: value 20K -> 1K
- TP4: renamed from TP8; footprint TestPoint:TestPoint_Pad_D1.5mm -> TestPoint:TestPoint_Pad_D2.5mm
- TP6, TP7: footprint TestPoint:TestPoint_Pad_D1.5mm -> TestPoint:TestPoint_Pad_D2.5mm
Connections:
- net labels added: GNDA
- wire segments 39 -> 54
- no-connect marks 3 -> 0
Other:
- moved on the sheet: C16, C18, D4, L2, Q1, Q2, R20, TP4, TP6, TP7

Commit message: This rev removes the safety micro and instead uses the dji battery
Parts:
- added Q5: DMG2301L, Package_TO_SOT_SMD:SOT-23, symbol Transistor_FET:DMG2301L
- IC8: symbol SmallKat-v2-rescue:TPS40192DRCT-TPS40192DRCT -> SmallKat-v2-rescue:TPS40192DRCT-TPS40192DRCT-SmallKat-v2-rescue-SmallKat-v2-rescue
Changed lines of the file:
@@
 $Descr A4 11693 8268
 encoding utf-8
-Sheet 11 12
+Sheet 7 7
 Title ""
 Date ""
@@
 $EndComp
 $Comp
-L SmallKat-v2-rescue:TPS40192DRCT-TPS40192DRCT IC8
+L SmallKat-v2-rescue:TPS40192DRCT-TPS40192DRCT-SmallKat-v2-rescue-SmallKat-v2-rescue IC8
 U 1 1 5E883273
 P 5100 2900
@@
 	1    0    0    -1
 $EndComp
-Text HLabel 4500 2900 0    50   Input ~ 0
+Text HLabel 4300 2600 1    50   Input ~ 0
 EN
+$Comp
+L Transistor_FET:DMG2301L Q5
+U 1 1 5F65AE85
+P 4300 2800
+F 0 "Q5" V 4549 2800 50  0000 C CNN
+F 1 "DMG2301L" V 4640 2800 50  0000 C CNN
+F 2 "Package_TO_SOT_SMD:SOT-23" H 4500 2725 50  0001 L CIN
+F 3 "https://www.diodes.com/assets/Datasheets/DMG2301L.pdf" H 4300 2800 50  0001 L CNN
+	1    4300 2800
+	0    -1   1    0
+$EndComp
+$Comp
+L power:+BATT #PWR0104
+U 1 1 5F661942
+P 4100 2900
+F 0 "#PWR0104" H 4100 2750 50  0001 C CNN
+F 1 "+BATT" V 4115 3027 50  0000 L CNN
+F 2 "" H 4100 2900 50  0001 C CNN
+F 3 "" H 4100 2900 50  0001 C CNN
+	1    4100 2900
+	0    -1   -1   0
+$EndComp
 $EndSCHEMATC

Commit message: batt connector and all in the right place. has not been ordered, waiting for prev rev to be tested first
Parts:
- IC8: symbol SmallKat-v2-rescue:TPS40192DRCT-TPS40192DRCT-SmallKat-v2-rescue-SmallKat-v2-rescue -> SmallKat-v2-rescue:TPS40192DRCT-TPS40192DRCT-SmallKat-v2-rescue-SmallKat-v2-rescue-SmallKat-v2-rescue
Changed lines of the file:
@@
 $EndComp
 $Comp
-L SmallKat-v2-rescue:TPS40192DRCT-TPS40192DRCT-SmallKat-v2-rescue-SmallKat-v2-rescue IC8
+L SmallKat-v2-rescue:TPS40192DRCT-TPS40192DRCT-SmallKat-v2-rescue-SmallKat-v2-rescue-SmallKat-v2-rescue IC8
 U 1 1 5E883273
 P 5100 2900

Commit message: rev, pendingorder
Parts:
- removed Q5: DMG2301L, Package_TO_SOT_SMD:SOT-23, symbol Transistor_FET:DMG2301L
- removed R17: 100k, Resistor_SMD:R_0402_1005Metric, symbol Device:R
- IC8: symbol SmallKat-v2-rescue:TPS40192DRCT-TPS40192DRCT-SmallKat-v2-rescue-SmallKat-v2-rescue-SmallKat-v2-rescue -> SmallKat-v2-rescue:TPS40192DRCT-TPS40192DRCT-SmallKat-v2-rescue-SmallKat-v2-rescue-SmallKat-v2-rescue-SmallKat-v2-rescu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
- Q1, Q2: value BUK9M120-100EX -> BUK9M17-30EX / BUK7M10-40E
- R16: value 3.9k -> 12k
- TP4: value TestPoint -> 6V
- TP6: value TestPoint -> Batt+
- TP7: value TestPoint -> GND
Connections:
- net labels removed: EN
- wire segments 54 -> 53
- no-connect marks 0 -> 1

Commit message: g
Parts:
- IC3: renamed from IC8; symbol SmallKat-v2-rescue:TPS40192DRCT-TPS40192DRCT-SmallKat-v2-rescue-SmallKat-v2-rescue-SmallKat-v2-rescue-SmallKat-v2-rescue-SmallKat-v2-rescue-SmallKat-v2-rescue-SmallKat-v2-rescue -> SmallKat-v2-rescue:TPS40192DRCT-TPS40192DRCT-SmallKat-v2-rescue-SmallKat-v2-rescue-SmallKat-v2-rescue-SmallKat-v2-rescue-SmallKat-v2-rescue-SmallKat-v2-rescue-SmallKat-v2-rescue-SmallKat-v2-rescue-SmallKat-v2-rescue
- renumbered C10 to C24, C11 to C25, C12 to C26, C13 to C27, C14 to C28, C15 to C29, C16 to C30, C17 to C31, C18 to C32, C19 to C33, C20 to C34, C21 to C35, C22 to C36, D4 to D13, L2 to L3, Q1 to Q2, Q2 to Q3, R12 to R36, R13 to R37, R14 to R38, R15 to R39, R16 to R40, R18 to R41, R19 to R42, R20 to R43, TP7 to TP10, TP4 to TP11, TP6 to TP9

Commit message: rev ordered
Parts:
- IC3: symbol SmallKat-v2-rescue:TPS40192DRCT-TPS40192DRCT-SmallKat-v2-rescue-SmallKat-v2-rescue-SmallKat-v2-rescue-SmallKat-v2-rescue-SmallKat-v2-rescue-SmallKat-v2-rescue-SmallKat-v2-rescue-SmallKat-v2-rescue-SmallKat-v2-rescue -> SmallKat-v2-rescue:TPS40192DRCT-TPS40192DRCT-SmallKat-v2-rescue-SmallKat-v2-rescue-SmallKat-v2-rescue-SmallKat-v2-rescue-SmallKat-v2-rescue-SmallKat-v2-rescue-SmallKat-v2-rescue-SmallKat-v2-rescue-SmallKat-v2-rescue-SmallKat-v2-rescue
Changed lines of the file:
@@
 $EndComp
 $Comp
-L SmallKat-v2-rescue:TPS40192DRCT-TPS40192DRCT-SmallKat-v2-rescue-SmallKat-v2-rescue-SmallKat-v2-rescue-SmallKat-v2-rescue-SmallKat-v2-rescue-SmallKat-v2-rescue-SmallKat-v2-rescue-SmallKat-v2-rescue-SmallKat-v2-rescue IC3
+L SmallKat-v2-rescue:TPS40192DRCT-TPS40192DRCT-SmallKat-v2-rescue-SmallKat-v2-rescue-SmallKat-v2-rescue-SmallKat-v2-rescue-SmallKat-v2-rescue-SmallKat-v2-rescue-SmallKat-v2-rescue-SmallKat-v2-rescue-SmallKat-v2-rescue-SmallKat-v2-rescue IC3
 U 1 1 5E883273
 P 5100 2900
