File: 3.sch (KiCad schematic (older format))
At the start: 22 parts, among them IC1 TPS562201DDCR, U2 LM2840Y

Commit message: Updated footprints
Parts:
- IC1: symbol TPS562201DDCR:TPS562201DDCR -> SmallKat-v2-rescue:TPS562201DDCR-TPS562201DDCR
Changed lines of the file:
@@
 EESchema Schematic File Version 4
-LIBS:SmallKat v2-cache
 EELAYER 30 0
 EELAYER END
@@
 $EndComp
 $Comp
-L TPS562201DDCR:TPS562201DDCR IC?
+L SmallKat-v2-rescue:TPS562201DDCR-TPS562201DDCR IC?
 U 1 1 5DAB2074
 P 6700 1200
