File: 3.sch (KiCad schematic (older format))
At the start: 22 parts, among them IC1 TPS562201DDCR, U2 LM2840Y

Commit message: Routing done
Parts:
- TP5: footprint TestPoint:TestPoint_Pad_D2.5mm -> TestPoint:TestPoint_Pad_D1.5mm
Connections:
- net labels added: +3.3VA
Changed lines of the file:
@@
 $Descr A4 11693 8268
 encoding utf-8
-Sheet 3 14
+Sheet 3 12
 Title ""
 Date ""
@@
 F 0 "TP5" H 7358 2318 50  0000 L CNN
 F 1 "TestPoint" H 7358 2227 50  0000 L CNN
-F 2 "TestPoint:TestPoint_Pad_D2.5mm" H 7500 2200 50  0001 C CNN
+F 2 "TestPoint:TestPoint_Pad_D1.5mm" H 7500 2200 50  0001 C CNN
 F 3 "~" H 7500 2200 50  0001 C CNN
 	1    7300 2200
@@
 Text HLabel 8200 1300 2    50   Input ~ 0
 EN
+$Comp
+L power:+3.3VA #PWR0116
+U 1 1 5DE1EB22
+P 4100 1000
+F 0 "#PWR0116" H 4100 850 50  0001 C CNN
+F 1 "+3.3VA" H 4115 1173 50  0000 C CNN
+F 2 "" H 4100 1000 50  0001 C CNN
+F 3 "" H 4100 1000 50  0001 C CNN
+	1    4100 1000
+	1    0    0    -1
+$EndComp
+Connection ~ 4100 1000
 $EndSCHEMATC

Commit message: order
Parts:
- removed D17: MA2YD26, Diode_SMD:D_SOD-123F, symbol Device:D
- removed U2: LM2840Y, Package_TO_SOT_SMD:TSOT-23-6, symbol Regulator_Switching:LM2840Y
- added C30, C34: 22uF, Capacitor_SMD:C_0805_2012Metric, symbol Device:C
- added C33: 0.1uF, Capacitor_SMD:C_0402_1005Metric, symbol Device:C
- added IC3: TPS562201DDCR, Package_TO_SOT_SMD:SOT-23-6, symbol SmallKat-v2-rescue:TPS562201DDCR-TPS562201DDCR
- added R28: 10K, Resistor_SMD:R_0402_1005Metric, symbol Device:R
- C23: value 2.2uF -> 10uF
- C25: value 0.1uF -> 10uF; footprint Capacitor_SMD:C_0402_1005Metric -> Capacitor_SMD:C_0805_2012Metric
- C35: value 10uF -> 0.1uF; footprint Capacitor_SMD:C_0805_2012Metric -> Capacitor_SMD:C_0402_1005Metric
- IC1: footprint TPS562201DDCR:SOT95P280X110-6N -> Package_TO_SOT_SMD:SOT-23-6; symbol TPS562201DDCR:TPS562201DDCR -> SmallKat-v2-rescue:TPS562201DDCR-TPS562201DDCR
- L3: value 15uH -> 4.7uH; footprint Inductor_SMD:L_1210_3225Metric -> Inductor_SMD:L_0805_2012Metric
- R2: value 1K -> 10K
- R3: value 3.4K -> 33.2K
Connections:
- net labels removed: VBUS
- wire segments 34 -> 32
Other:
- moved on the sheet: C1, C2, C3, C4, C5, C6, D3, L1, R10, R7, R8, R9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

Commit message: This rev removes the safety micro and instead uses the dji battery
Parts:
- removed C34: 22uF, Capacitor_SMD:C_0805_2012Metric, symbol Device:C
- removed C35: 0.1uF, Capacitor_SMD:C_0402_1005Metric, symbol Device:C
- removed IC3: TPS562201DDCR, Package_TO_SOT_SMD:SOT-23-6, symbol SmallKat-v2-rescue:TPS562201DDCR-TPS562201DDCR
- removed R2: 10K, Resistor_SMD:R_0402_1005Metric, symbol Device:R
- removed R3: 33.2K, Resistor_SMD:R_0402_1005Metric, symbol Device:R
- added C20, C22: 10uF, Capacitor_SMD:C_0805_2012Metric, symbol Device:C
- added IC2: TPS562201DDCR, Package_TO_SOT_SMD:SOT-23-6, symbol SmallKat-v2-rescue:TPS562201DDCR-TPS562201DDCR-SmallKat-v2-rescue-SmallKat-v2-r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
- added R29: 33.2K, Resistor_SMD:R_0402_1005Metric, symbol Device:R
- added R30: 10K, Resistor_SMD:R_0402_1005Metric, symbol Device:R
- C23: value 10uF -> 22uF
- C25: value 10uF -> 0.1uF; footprint Capacitor_SMD:C_0805_2012Metric -> Capacitor_SMD:C_0402_1005Metric
- IC1: symbol SmallKat-v2-rescue:TPS562201DDCR-TPS562201DDCR -> SmallKat-v2-rescue:TPS562201DDCR-TPS562201DDCR-SmallKat-v2-rescue-SmallKat-v2-rescue
Connections:
- net labels added: VBUS
- net labels removed: +3.3VA, EN

Commit message: batt connector and all in the right place. has not been ordered, waiting for prev rev to be tested first
Parts:
- added D5, D6: DIODE, Diode_SMD:D_SOD-123F, symbol pspice:DIODE
- IC1, IC2: symbol SmallKat-v2-rescue:TPS562201DDCR-TPS562201DDCR-SmallKat-v2-rescue-SmallKat-v2-rescue -> SmallKat-v2-rescue:TPS562201DDCR-TPS562201DDCR-SmallKat-v2-rescue-SmallKat-v2-rescue-SmallKat-v2-rescue
Changed lines of the file:
@@
 $EndComp
 $Comp
-L SmallKat-v2-rescue:TPS562201DDCR-TPS562201DDCR-SmallKat-v2-rescue-SmallKat-v2-rescue IC?
+L SmallKat-v2-rescue:TPS562201DDCR-TPS562201DDCR-SmallKat-v2-rescue-SmallKat-v2-rescue-SmallKat-v2-rescue IC?
 U 1 1 5DAB2074
 P 2550 1050
@@
 L power:+3.3V #PWR?
 U 1 1 5DAB20BF
-P 1350 1150
+P 950 1150
 AR Path="/5DAB20BF" Ref="#PWR?"  Part="1"
 AR Path="/5DAA9390/5DAAD545/5DAB20BF" Ref="#PWR0136"  Part="1"
-F 0 "#PWR0136" H 1350 1000 50  0001 C CNN
-F 1 "+3.3V" V 1365 1278 50  0000 L CNN
-F 2 "" H 1350 1150 50  0001 C CNN
-F 3 "" H 1350 1150 50  0001 C CNN
-	1    1350 1150
+F 0 "#PWR0136" H 950 1000 50  0001 C CNN
+F 1 "+3.3V" V 965 1278 50  0000 L CNN
+F 2 "" H 950 1150 50  0001 C CNN
+F 3 "" H 950 1150 50  0001 C CNN
+	1    950  1150
 	0    -1   -1   0
 $EndComp
@@
 $EndComp
 $Comp
-L SmallKat-v2-rescue:TPS562201DDCR-TPS562201DDCR-SmallKat-v2-rescue-SmallKat-v2-rescue IC?
+L SmallKat-v2-rescue:TPS562201DDCR-TPS562201DDCR-SmallKat-v2-rescue-SmallKat-v2-rescue-SmallKat-v2-rescue IC?
 U 1 1 5FB8C063
 P 2550 2750
@@
 L power:+3.3V #PWR?
 U 1 1 5FB8C0A7
-P 1350 2850
+P 950 2850
 AR Path="/5FB8C0A7" Ref="#PWR?"  Part="1"
 AR Path="/5DAA9390/5DAAD545/5FB8C0A7" Ref="#PWR0153"  Part="1"
 AR Path="/5DAA9390/5DAAB924/5FB8C0A7" Ref="#PWR?"  Part="1"
-F 0 "#PWR0153" H 1350 2700 50  0001 C CNN
-F 1 "+3.3V" V 1365 2978 50  0000 L CNN
-F 2 "" H 1350 2850 50  0001 C CNN
-F 3 "" H 1350 2850 50  0001 C CNN
-	1    1350 2850
+F 0 "#PWR0153" H 950 2700 50  0001 C CNN
+F 1 "+3.3V" V 965 2978 50  0000 L CNN
+F 2 "" H 950 2850 50  0001 C CNN
+F 3 "" H 950 2850 50  0001 C CNN
+	1    950  2850
 	0    -1   -1   0
 $EndComp
@@
 Wire Wire Line
 	1200 3150 1550 3150
-$Comp
-L power:+BATT #PWR0174
-U 1 1 5FB8C0B4
-P 4050 2850
-AR Path="/5DAA9390/5DAAD545/5FB8C0B4" Ref="#PWR0174"  Part="1"
-AR Path="/5DAA9390/5DAAB924/5FB8C0B4" Ref="#PWR?"  Part="1"
-F 0 "#PWR0174" H 4050 2700 50  0001 C CNN
-F 1 "+BATT" V 4065 2977 50  0000 L CNN
-F 2 "" H 4050 2850 50  0001 C CNN
-F 3 "" H 4050 2850 50  0001 C CNN
-	1    4050 2850
-	0    1    -1   0
-$EndComp
 $Comp
 L power:VBUS #PWR?
@@
 $EndComp
 Connection ~ 1200 3450
+$Comp
+L pspice:DIODE D5
+U 1 1 5FC888B1
+P 1150 1150
+F 0 "D5" H 1150 885 50  0000 C CNN
+F 1 "DIODE" H 1150 976 50  0000 C CNN
+F 2 "Diode_SMD:D_SOD-123F" H 1150 1150 50  0001 C CNN
+F 3 "~" H 1150 1150 50  0001 C CNN
+	1    1150 1150
+	-1   0    0    1
+$EndComp
+$Comp
+L pspice:DIODE D6
+U 1 1 5FC895A5
+P 1150 2850
+F 0 "D6" H 1150 2585 50  0000 C CNN
+F 1 "DIODE" H 1150 2676 50  0000 C CNN
+F 2 "Diode_SMD:D_SOD-123F" H 1150 2850 50  0001 C CNN
+F 3 "~" H 1150 2850 50  0001 C CNN
+	1    1150 2850
+	-1   0    0    1
+$EndComp
+$Comp
+L power:VBUS #PWR?
+U 1 1 5FC87AF3
+P 4050 2850
+AR Path="/5DAA9390/5DAAB924/5FC87AF3" Ref="#PWR?"  Part="1"
+AR Path="/5DAA9E7A/5DB7E2D8/5FC87AF3" Ref="#PWR?"  Part="1"
+AR Path="/5DAA9390/5DAAD545/5FC87AF3" Ref="#PWR?"  Part="1"
+F 0 "#PWR?" H 4050 2700 50  0001 C CNN
+F 1 "VBUS" H 4065 3023 50  0000 C CNN
+F 2 "" H 4050 2850 50  0001 C CNN
+F 3 "" H 4050 2850 50  0001 C CNN
+	1    4050 2850
+	0    1    1    0
+$EndComp
 $EndSCHEMATC

Commit message: rev, pendingorder
Parts:
- IC1, IC2: symbol SmallKat-v2-rescue:TPS562201DDCR-TPS562201DDCR-SmallKat-v2-rescue-SmallKat-v2-rescue-SmallKat-v2-rescue -> SmallKat-v2-rescue:TPS562201DDCR-TPS562201DDCR-SmallKat-v2-rescue-SmallKat-v2-rescue-SmallKat-v2-rescue-SmallKat-v2-res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
- TP5: value TestPoint -> 3.3v

Commit message: g
Parts:
- IC1, IC2: symbol SmallKat-v2-rescue:TPS562201DDCR-TPS562201DDCR-SmallKat-v2-rescue-SmallKat-v2-rescue-SmallKat-v2-rescue-SmallKat-v2-rescue-SmallKat-v2-rescue-SmallKat-v2-rescue-SmallKat-v2-rescue -> SmallKat-v2-rescue:TPS562201DDCR-TPS562201DDCR-SmallKat-v2-rescue-SmallKat-v2-rescue-SmallKat-v2-rescue-SmallKat-v2-rescue-SmallKat-v2-rescue-SmallKat-v2-rescue-SmallKat-v2-rescue-SmallKat-v2-rescue-SmallKat-v2-rescue
- renumbered C5 to C10, C30 to C11, C6 to C12, C33 to C13, C1 to C2, C20 to C3, C2 to C4, C22 to C5, C3 to C6, C23 to C7, C4 to C8, C25 to C9, D5 to D4, D6 to D5, D3 to D6, L3 to L2, R8 to R10, R28 to R11, R9 to R12, R29 to R13, R10 to R14, R30 to R15, R7 to R16, TP5 to TP4

Commit message: rev ordered
Parts:
- removed C10, C11, C7: 22uF, Capacitor_SMD:C_0805_2012Metric, symbol Device:C
- removed C13, C8, C9: 0.1uF, Capacitor_SMD:C_0402_1005Metric, symbol Device:C
- removed IC1, IC2: TPS562201DDCR, Package_TO_SOT_SMD:SOT-23-6, symbol SmallKat-v2-rescue:TPS562201DDCR-TPS562201DDCR-SmallKat-v2-rescue-SmallKat-v2-r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
- removed R14, R15: 10K, Resistor_SMD:R_0402_1005Metric, symbol Device:R
- added F6, F7: Fuse, Fuse:Fuse_1210_3225Metric, symbol Device:Fuse
- added IC1, IC2: LMR14010A, Package_TO_SOT_SMD:SOT-23-6, symbol LMR50410YQDBVRQ1:LMR50410YQDBVRQ1
- C2, C5: value 10uF -> 2.2uF
- C3: value 10uF -> 0.1uF; footprint Capacitor_SMD:C_0805_2012Metric -> Capacitor_SMD:C_0402_1005Metric
- C6: value 22uF -> 10uF
- L1, L2: value 4.7uH -> 10uH
- R11: value 10K -> 33.2
- R12: value 33.2K -> 33.2
- R13: value 33.2K -> 10K
Connections:
- wire segments 32 -> 18
Other:
- moved on the sheet: C12, C2, C4, D4, L1, R10, R12

Commit message: ordered version with foot connecotrs
Parts:
- F6, F7: footprint Fuse:Fuse_1210_3225Metric -> Fuse:Fuse_1206_3216Metric
Changed lines of the file:
@@
 F 0 "F6" V 7603 1250 50  0000 C CNN
 F 1 "Fuse" V 7694 1250 50  0000 C CNN
-F 2 "Fuse:Fuse_1210_3225Metric" V 7730 1250 50  0001 C CNN
+F 2 "Fuse:Fuse_1206_3216Metric" V 7730 1250 50  0001 C CNN
 F 3 "~" H 7800 1250 50  0001 C CNN
 	1    7800 1250
@@
 F 0 "F7" V 7753 2700 50  0000 C CNN
 F 1 "Fuse" V 7844 2700 50  0000 C CNN
-F 2 "Fuse:Fuse_1210_3225Metric" V 7880 2700 50  0001 C CNN
+F 2 "Fuse:Fuse_1206_3216Metric" V 7880 2700 50  0001 C CNN
 F 3 "~" H 7950 2700 50  0001 C CNN
 	1    7950 2700
