File: BatteryBalancer.sch (KiCad schematic (older format))
At the start: 14 parts, among them J21 Conn_01x05_Male, U13 bq76925

Commit message: Updated footprints
Parts:
- U13: symbol bq76925:bq76925 -> SmallKat-v2-rescue:bq76925-bq76925
Changed lines of the file:
@@
 EESchema Schematic File Version 4
-LIBS:SmallKat v2-cache
 EELAYER 30 0
 EELAYER END
@@
 $EndDescr
 $Comp
-L bq76925:bq76925 U13
+L SmallKat-v2-rescue:bq76925-bq76925 U13
 U 1 1 5DD78636
 P 5000 3450
