File: BatteryBalancer.sch (KiCad schematic (older format))
At the start: 14 parts, among them J21 Conn_01x05_Male, U13 bq76925

Commit message: order
Parts:
- U13: symbol bq76925:bq76925 -> SmallKat-v2-rescue:bq76925-bq76925
Changed lines of the file:
@@
 EESchema Schematic File Version 4
-LIBS:SmallKat v2-cache
 EELAYER 30 0
 EELAYER END
 $Descr A4 11693 8268
 encoding utf-8
-Sheet 12 12
+Sheet 11 12
 Title ""
 Date ""
@@
 $EndDescr
 $Comp
-L bq76925:bq76925 U13
+L SmallKat-v2-rescue:bq76925-bq76925 U13
 U 1 1 5DD78636
 P 5000 3450
+AR Path="/5DD78636" Ref="U13"  Part="1"
+AR Path="/5DAA9390/5DD78452/5DD78636" Ref="U13"  Part="1"
 F 0 "U13" H 5744 3471 50  0000 L CNN
 F 1 "bq76925" H 5744 3380 50  0000 L CNN

Commit message: This rev removes the safety micro and instead uses the dji battery
Parts:
- U13: symbol SmallKat-v2-rescue:bq76925-bq76925 -> SmallKat-v2-rescue:bq76925-bq76925-SmallKat-v2-rescue
Changed lines of the file:
@@
 $EndDescr
 $Comp
-L SmallKat-v2-rescue:bq76925-bq76925 U13
+L SmallKat-v2-rescue:bq76925-bq76925-SmallKat-v2-rescue U13
 U 1 1 5DD78636
 P 5000 3450
