File: BatteryCharging.sch (KiCad schematic (older format))
At the start: 52 parts, among them Q10 CSD17307Q5A, Q11 CSD17307Q5A, Q12 Si7141DP, Q8 BUK9M120-100EX, Q9 BUK9M120-100EX, U12 BQ24770

Commit message: Rev
Parts:
- C69, C74: footprint Capacitor_SMD:C_0402_1005Metric -> Capacitor_SMD:C_0805_2012Metric
- R123: footprint Resistor_SMD:R_0603_1608Metric -> Resistor_SMD:R_0805_2012Metric
Changed lines of the file:
@@
 F 0 "C69" H 9065 1696 50  0000 L CNN
 F 1 "10uF" H 9065 1605 50  0000 L CNN
-F 2 "Capacitor_SMD:C_0402_1005Metric" H 8988 1500 50  0001 C CNN
+F 2 "Capacitor_SMD:C_0805_2012Metric" H 8988 1500 50  0001 C CNN
 F 3 "~" H 8950 1650 50  0001 C CNN
 	1    8950 1650
@@
 F 0 "R123" V 9093 1500 50  0000 C CNN
 F 1 "0.01R" V 9184 1500 50  0000 C CNN
-F 2 "Resistor_SMD:R_0603_1608Metric" V 9230 1500 50  0001 C CNN
+F 2 "Resistor_SMD:R_0805_2012Metric" V 9230 1500 50  0001 C CNN
 F 3 "~" H 9300 1500 50  0001 C CNN
 	1    9300 1500
@@
 F 0 "C74" H 9815 1696 50  0000 L CNN
 F 1 "10uF" H 9815 1605 50  0000 L CNN
-F 2 "Capacitor_SMD:C_0402_1005Metric" H 9738 1500 50  0001 C CNN
+F 2 "Capacitor_SMD:C_0805_2012Metric" H 9738 1500 50  0001 C CNN
 F 3 "~" H 9700 1650 50  0001 C CNN
 	1    9700 1650
