File: BatteryCharging.sch (KiCad schematic (older format))
At the start: 52 parts, among them Q10 CSD17307Q5A, Q11 CSD17307Q5A, Q12 Si7141DP, Q8 BUK9M120-100EX, Q9 BUK9M120-100EX, U12 BQ24770

Commit message: This rev removes the safety micro and instead uses the dji battery
Parts:
- Q12: symbol SmallKat-v2-rescue:Si7141DP-Transistor_FET -> SmallKat-v2-rescue:Si7141DP-Transistor_FET-SmallKat-v2-rescue
- U12: symbol SmallKat-v2-rescue:BQ24770-BQ24770 -> SmallKat-v2-rescue:BQ24770-BQ24770-SmallKat-v2-rescue
Changed lines of the file:
@@
 $EndDescr
 $Comp
-L SmallKat-v2-rescue:BQ24770-BQ24770 U12
+L SmallKat-v2-rescue:BQ24770-BQ24770-SmallKat-v2-rescue U12
 U 1 1 5DD6E3BB
 P 5750 2550
+AR Path="/5DD6E3BB" Ref="U12"  Part="1"
+AR Path="/5DAA9390/5DD4BDB9/5DD6E3BB" Ref="U12"  Part="1"
 F 0 "U12" H 6400 2050 50  0000 C CNN
 F 1 "BQ24770" H 6450 1900 50  0000 C CNN
@@
 $EndComp
 $Comp
-L SmallKat-v2-rescue:Si7141DP-Transistor_FET Q12
+L SmallKat-v2-rescue:Si7141DP-Transistor_FET-SmallKat-v2-rescue Q12
 U 1 1 5DDBB55A
 P 10250 1600
