File: SafetyMCU.sch (KiCad schematic (older format))
At the start: 18 parts, among them Q7 2N3905, SW5 SW_SPST, U6 STM32L432KBUx

Commit message: order
Parts:
- added D6: LED, LED_SMD:LED_0603_1608Metric, symbol Device:LED
- added R31: 330R, Resistor_SMD:R_0402_1005Metric, symbol Device:R
Connections:
- net GND: now also D6.1 (K)
- net at U6.18 (PA8): now also R31.2
- new net: D6.2 (A), R31.1
Changed lines of the file:
@@
 EESchema Schematic File Version 4
-LIBS:SmallKat v2-cache
 EELAYER 30 0
 EELAYER END
 $Descr A4 11693 8268
 encoding utf-8
-Sheet 7 12
+Sheet 6 12
 Title ""
 Date ""
@@
 $EndComp
 $Comp
-L power:+3.3VA #PWR?
+L power:+3.3VA #PWR0198
 U 1 1 5DE37C49
 P 4000 2300
-F 0 "#PWR?" H 4000 2150 50  0001 C CNN
+F 0 "#PWR0198" H 4000 2150 50  0001 C CNN
 F 1 "+3.3VA" H 4015 2473 50  0000 C CNN
 F 2 "" H 4000 2300 50  0001 C CNN
@@
 	-1   0    0    1
 $EndComp
+$Comp
+L Device:R R31
+U 1 1 5E0D8EE1
+P 2650 2150
+F 0 "R31" V 2443 2150 50  0000 C CNN
+F 1 "330R" V 2534 2150 50  0000 C CNN
+F 2 "Resistor_SMD:R_0402_1005Metric" V 2580 2150 50  0001 C CNN
+F 3 "~" H 2650 2150 50  0001 C CNN
+	1    2650 2150
+	0    1    1    0
+$EndComp
+$Comp
+L Device:LED D6
+U 1 1 5E0D93B9
+P 2950 2150
+F 0 "D6" H 2943 1895 50  0000 C CNN
+F 1 "LED" H 2943 1986 50  0000 C CNN
+F 2 "LED_SMD:LED_0603_1608Metric" H 2950 2150 50  0001 C CNN
+F 3 "~" H 2950 2150 50  0001 C CNN
+	1    2950 2150
+	-1   0    0    1
+$EndComp
+$Comp
+L power:GND #PWR0202
+U 1 1 5E0D991B
+P 3100 2150
+F 0 "#PWR0202" H 3100 1900 50  0001 C CNN
+F 1 "GND" H 3105 1977 50  0000 C CNN
+F 2 "" H 3100 2150 50  0001 C CNN
+F 3 "" H 3100 2150 50  0001 C CNN
+	1    3100 2150
+	1    0    0    -1
+$EndComp
 $EndSCHEMATC
