File: SafetyMCU.sch (KiCad schematic (older format))
At the start: 20 parts, among them Q7 2N3905, SW5 SW_SPST, U6 STM32L432KBUx

Commit message: Rev
Parts:
- removed C37, C45, C46: 0.1uF, Capacitor_SMD:C_0402_1005Metric, symbol Device:C
- removed R43: 10K, Resistor_SMD:R_0402_1005Metric, symbol Device:R
- removed U6: STM32L432KBUx, Package_DFN_QFN:QFN-32-1EP_5x5mm_P0.5mm_EP3.45x3.45mm, symbol MCU_ST_STM32L4:STM32L432KBUx
- added C22, C36: C, Capacitor_SMD:C_0402_1005Metric, symbol Device:C
- added TP8: TestPoint, TestPoint:TestPoint_Pad_D1.5mm, symbol Connector:TestPoint
- added U5: LPC824M201JHI33, Package_DFN_QFN:QFN-32-1EP_5x5mm_P0.5mm_EP3.45x3.45mm, symbol MCU_NXP_LPC:LPC824M201JHI33
Connections:
- net +3.3VA: now also C22.2, C36.2, U5.19 (VDD), U5.21 (VREFP)
- net 3.3VEN: now also U5.28 (PIO0_21)
- net 6VEN: now also U5.29 (PIO0_20)
- net BUZZER: now also U5.18 (PIO0_8)
- net GND: now also C22.1, C36.1, U5.20 (VREFN), U5.33 (VSS)
- net MONITORING: now also U5.25 (PIO0_14)
- net NRST: now also TP8.1, U5.3 (PIO0_5)
- net SCL: now also U5.31 (PIO0_18); no longer R45.2
- net SDA: now also U5.32 (PIO0_17); no longer R46.2
- net SOFTPOWER: now also U5.11 (PIO0_27)
- net at R31.2: now also U5.8 (PIO0_11)
- net at TP20.1: now also U5.7 (PIO0_2)
- net at TP21.1: now also U5.6 (PIO0_3)
- new net I2CTALKALLOWED: U5.2 (PIO0_12)
- new net I2CTALKING: U5.1 (PIO0_13)
- new net RX: U5.24 (PIO0_0)
- new net SCL1: R45.2, U5.27 (PIO0_22)
- new net SDA1: R46.2, U5.26 (PIO0_23)
- new net TX: U5.4 (PIO0_4)
Other:
- moved on the sheet: D6, R31, R46, TP20, TP21
