File: i2cArbiter.sch (KiCad schematic (older format))
At the start: 4 parts, among them U14 PCA9641

Commit message: order
Parts:
- U14: symbol PCA9641:PCA9641 -> SmallKat-v2-rescue:PCA9641-PCA9641
Changed lines of the file:
@@
 EESchema Schematic File Version 4
-LIBS:SmallKat v2-cache
 EELAYER 30 0
 EELAYER END
@@
 $EndDescr
 $Comp
-L PCA9641:PCA9641 U14
+L SmallKat-v2-rescue:PCA9641-PCA9641 U14
 U 1 1 5DD9F97C
 P 4750 3450
