File: MainBoard.sch (KiCad schematic (older format))
At the start: 12 parts, among them J9 Conn_01x02_Male

Commit message: order
Changed lines of the file:
@@
 EESchema Schematic File Version 4
-LIBS:SmallKat v2-cache
 EELAYER 30 0
 EELAYER END
@@
 F2 "SDA" I L 7950 4900 50
 F3 "SCL" I L 7950 5100 50
-$EndSheet
-$Sheet
-S 7250 650  1750 1550
-U 5DAC8B3A
-F0 "6vSwitchMode" 50
-F1 "6vSwitchMode.sch" 50
-F2 "EN" I L 7250 1400 50
 $EndSheet
 $Comp
@@
 Text Label 7250 2950 2    50   ~ 0
 3.3VEN
-Text Label 7250 1400 2    50   ~ 0
-6VEN
 Text Label 9550 1400 2    50   ~ 0
 3.3VEN
@@
 Wire Wire Line
 	1350 1950 1850 1950
+$Sheet
+S 7250 700  1750 1550
+U 5E0C112B
+F0 "sheet5E0C1128" 50
+F1 "6vSwitchMode.sch" 50
+F2 "EN" I L 7250 1450 50
+$EndSheet
+Text Label 7250 1450 2    50   ~ 0
+6VEN
 $EndSCHEMATC

Commit message: Rev
Parts:
- H1, H2, H3, H4: footprint MountingHole:MountingHole_2.7mm_M2.5_Pad_Via -> MountingHole:MountingHole_3.2mm_M3_Pad_Via
- J9: footprint SmallKat ESP32:SHDR2W320P716_1X2_1574X813X1588P -> XT30PB:XT30PB
Connections:
- net labels added: NRST, RX1, SERVO16, SERVO17, SERVO18, SERVO19, TALKALLOWED, TALKING, TX1
- net labels removed: _SCL, _SDA
- wire segments 9 -> 8
Changed lines of the file:
@@
 $EndDescr
 $Sheet
-S 9550 700  1450 1400
+S 7250 1150 550  300
 U 5DAAD545
 F0 "3.3v Switchmode" 50
 F1 "3.sch" 50
-F2 "EN" I L 9550 1400 50
+F2 "EN" I L 7250 1300 50
 $EndSheet
 $Comp
@@
 F 0 "H3" H 5100 6749 50  0000 L CNN
 F 1 "MountingHole_Pad" H 5100 6658 50  0000 L CNN
-F 2 "MountingHole:MountingHole_2.7mm_M2.5_Pad_Via" H 5000 6700 50  0001 C CNN
+F 2 "MountingHole:MountingHole_3.2mm_M3_Pad_Via" H 5000 6700 50  0001 C CNN
 F 3 "~" H 5000 6700 50  0001 C CNN
 	1    5000 6700
@@
 F 0 "H1" H 4800 6749 50  0000 L CNN
 F 1 "MountingHole_Pad" H 4800 6658 50  0000 L CNN
-F 2 "MountingHole:MountingHole_2.7mm_M2.5_Pad_Via" H 4700 6700 50  0001 C CNN
+F 2 "MountingHole:MountingHole_3.2mm_M3_Pad_Via" H 4700 6700 50  0001 C CNN
 F 3 "~" H 4700 6700 50  0001 C CNN
 	1    4700 6700
@@
 F 0 "H4" H 5100 7249 50  0000 L CNN
 F 1 "MountingHole_Pad" H 5100 7158 50  0000 L CNN
-F 2 "MountingHole:MountingHole_2.7mm_M2.5_Pad_Via" H 5000 7200 50  0001 C CNN
+F 2 "MountingHole:MountingHole_3.2mm_M3_Pad_Via" H 5000 7200 50  0001 C CNN
 F 3 "~" H 5000 7200 50  0001 C CNN
 	1    5000 7200
@@
 F 0 "H2" H 4800 7249 50  0000 L CNN
 F 1 "MountingHole_Pad" H 4800 7158 50  0000 L CNN
-F 2 "MountingHole:MountingHole_2.7mm_M2.5_Pad_Via" H 4700 7200 50  0001 C CNN
+F 2 "MountingHole:MountingHole_3.2mm_M3_Pad_Via" H 4700 7200 50  0001 C CNN
 F 3 "~" H 4700 7200 50  0001 C CNN
 	1    4700 7200
@@
 $EndComp
 $Sheet
-S 7950 4550 900  950
+S 7900 4300 900  950
 U 5DAC4399
 F0 "BNO055" 50
 F1 "BNO055.sch" 50
-F2 "SDA" I L 7950 4900 50
-F3 "SCL" I L 7950 5100 50
+F2 "SDA" I L 7900 4650 50
+F3 "SCL" I L 7900 4850 50
 $EndSheet
 $Comp
@@
 F 0 "J9" V 1060 7040 50  0000 L CNN
 F 1 "Conn_01x02_Male" V 1151 7040 50  0000 L CNN
-F 2 "SmallKat ESP32:SHDR2W320P716_1X2_1574X813X1588P" H 1000 7000 50  0001 C CNN
+F 2 "XT30PB:XT30PB" H 1000 7000 50  0001 C CNN
 F 3 "~" H 1000 7000 50  0001 C CNN
 	1    1000 7000
@@
 Wire Wire Line
 	1700 2950 1850 2950
-Text Label 7800 5100 2    50   ~ 0
+Text Label 7750 4850 2    50   ~ 0
 SCL
 Wire Wire Line
-	7800 5100 7950 5100
-Text Label 7800 4900 2    50   ~ 0
+	7750 4850 7900 4850
+Text Label 7750 4650 2    50   ~ 0
 SDA
 Wire Wire Line
-	7800 4900 7950 4900
+	7750 4650 7900 4650
 $Sheet
 S 1850 800  1600 2600
@@
 F24 "CC2" I L 1850 3200 50
 $EndSheet
-Text Label 1850 1050 2    50   ~ 0
-SERVO14
-Text Label 1850 1750 2    50   ~ 0
-SERVO15
-Text Label 1850 950  2    50   ~ 0
-SERVO11
-Text Label 1850 1650 2    50   ~ 0
-SERVO13
 $Comp
 L Device:R R6
@@
 	1    0    0    -1
 $EndComp
-Text Label 1850 850  2    50   ~ 0
-SERVO10
-Text Label 1250 1250 2    50   ~ 0
-SERVO8
-Text Label 1850 1150 2    50   ~ 0
-SERVO0
-Text Label 1850 1350 2    50   ~ 0
-SERVO1
-Text Label 1850 2250 2    50   ~ 0
-SERVO2
-Text Label 1850 2150 2    50   ~ 0
-SERVO3
-Text Label 1850 2050 2    50   ~ 0
-SERVO4
-Text Label 1850 2450 2    50   ~ 0
-SERVO5
-Text Label 1850 2350 2    50   ~ 0
-SERVO6
-Text Label 1850 1450 2    50   ~ 0
-SERVO9
 $Comp
 L Connector:TestPoint TP2
@@
 Text Label 5000 1050 3    50   ~ 0
 SCL
-Text Label 1850 1850 2    50   ~ 0
-SERVO7
-Text Label 1850 1550 2    50   ~ 0
-SERVO12
 $Comp
 L Device:R R1
@@
 F4 "SCL" I L 7250 3100 50
 F5 "SDA" I L 7250 3200 50
-$EndSheet
-$Sheet
-S 9800 4650 1100 550
+F6 "NRST" I L 7250 3350 50
+F7 "TX" I L 7250 3450 50
+F8 "RX" I L 7250 3550 50
+F9 "I2CTALKALLOWED" I L 7250 3650 50
+F10 "I2CTALKING" I L 7250 3750 50
+F11 "SCL1" I L 7250 3850 50
+F12 "SDA1" I L 7250 3950 50
+$EndSheet
+$Sheet
+S 9800 5000 1100 550
 U 5DD4BD78
 F0 "USBPD" 50
 F1 "USBPD.sch" 50
-F2 "CC1" I L 9800 4750 50
-F3 "CC2" I L 9800 4850 50
-F4 "SCL" I L 9800 4950 50
-F5 "SDA" I L 9800 5050 50
-$EndSheet
-$Sheet
-S 9800 5450 1100 650
+F2 "CC1" I L 9800 5100 50
+F3 "CC2" I L 9800 5200 50
+F4 "SCL" I L 9800 5300 50
+F5 "SDA" I L 9800 5400 50
+$EndSheet
+$Sheet
+S 9800 5800 1100 650
 U 5DD4BDB9
 F0 "Sheet5DD4BDB8" 50
 F1 "BatteryCharging.sch" 50
-F2 "SDA" I L 9800 5600 50
-F3 "SCL" I L 9800 5700 50
-$EndSheet
-$Sheet
-S 9750 2500 1200 1700
+F2 "SDA" I L 9800 5950 50
+F3 "SCL" I L 9800 6050 50
+$EndSheet
+$Sheet
+S 9750 2500 1200 2050
 U 5DD5998B
 F0 "Servos" 50
@@
 F18 "SERVO15" I L 9750 4000 50
 F19 "SERVO16" I L 9750 4100 50
-$EndSheet
-Text Label 7250 3100 2    50   ~ 0
+F20 "SERVO17" I L 9750 4200 50
+F21 "SERVO18" I L 9750 4300 50
+F22 "SERVO19" I L 9750 4400 50
+F23 "SERVO20" I L 9750 4500 50
+$EndSheet
+Text Label 9800 5300 2    50   ~ 0
 SAFETYSCL
-Text Label 7250 3200 2    50   ~ 0
+Text Label 9800 5400 2    50   ~ 0
 SAFETYSDA
-Text Label 9800 4950 2    50   ~ 0
-SAFETYSCL
-Text Label 9800 5050 2    50   ~ 0
-SAFETYSDA
-Text Label 9800 4850 2    50   ~ 0
+Text Label 9800 5200 2    50   ~ 0
 CC2
-Text Label 9800 4750 2    50   ~ 0
+Text Label 9800 5100 2    50   ~ 0
 CC1
 Text Label 1850 3200 2    50   ~ 0
@@
 	-1   0    0    1
 $EndComp
-Text Label 9800 5700 2    50   ~ 0
+Text Label 9800 6050 2    50   ~ 0
 SAFETYSCL
-Text Label 9800 5600 2    50   ~ 0
+Text Label 9800 5950 2    50   ~ 0
 SAFETYSDA
-Text Label 10950 2650 0    50   ~ 0
-_SDA
 Text Label 10950 2800 0    50   ~ 0
-_SCL
+SCL
 Text Label 9750 2600 2    50   ~ 0
 SERVO0
@@
 Text Label 7250 2950 2    50   ~ 0
 3.3VEN
-Text Label 9550 1400 2    50   ~ 0
+Text Label 7250 1300 2    50   ~ 0
 3.3VEN
 $Sheet
-S 6400 4450 950  950
-U 5DD78216
-F0 "i2cArbiter" 50
-F1 "i2cArbiter.sch" 50
-F2 "SCL1" I L 6400 4550 50
-F3 "SDA1" I L 6400 4650 50
-F4 "SCL2" I L 6400 4800 50
-F5 "SDA2" I L 6400 4900 50
-F6 "SCL_SLAVE" O L 6400 5100 50
-F7 "SDA_SLAVE" O L 6400 5200 50
-$EndSheet
-$Sheet
-S 5850 2750 800  950
+S 9800 750  800  950
 U 5DD78452
 F0 "BatteryBalancer" 50
 F1 "BatteryBalancer.sch" 50
-F2 "SCL" I L 5850 3100 50
-F3 "SDA" I L 5850 3200 50
-$EndSheet
-Text Label 6400 5200 2    50   ~ 0
-_SDA
-Text Label 6400 5100 2    50   ~ 0
-_SCL
-Text Label 6400 4800 2    50   ~ 0
-SAFETYSCL
-Text Label 6400 4900 2    50   ~ 0
-SAFETYSDA
-Text Label 6400 4650 2    50   ~ 0
+F2 "SCL" I L 9800 1100 50
+F3 "SDA" I L 9800 1200 50
+$EndSheet
+Text Label 7250 3200 2    50   ~ 0
 SDA
-Text Label 6400 4550 2    50   ~ 0
+Text Label 7250 3100 2    50   ~ 0
 SCL
-Text Label 5850 3100 2    50   ~ 0
-SAFETYSCL
-Text Label 5850 3200 2    50   ~ 0
-SAFETYSDA
-Wire Wire Line
-	1250 1250 1850 1250
-Wire Wire Line
-	1350 1950 1850 1950
-$Sheet
-S 7250 700  1750 1550
+$Sheet
+S 7250 700  550  250
 U 5E0C112B
 F0 "sheet5E0C1128" 50
 F1 "6vSwitchMode.sch" 50
-F2 "EN" I L 7250 1450 50
-$EndSheet
-Text Label 7250 1450 2    50   ~ 0
+F2 "EN" I L 7250 800 50
+$EndSheet
+Text Label 7250 800  2    50   ~ 0
 6VEN
+$Sheet
+S 3300 3750 850  2050
+U 5E683C3E
+F0 "PWMExpander" 50
+F1 "PWMExpandeR.sch" 50
+F2 "SCK" I L 3300 4000 50
+F3 "MOSI" I L 3300 4100 50
+F4 "SERVO0" O R 4150 3850 50
+F5 "SERVO1" O R 4150 3950 50
+F6 "SERVO2" O R 4150 4050 50
+F7 "SERVO3" O R 4150 4150 50
+F8 "SERVO4" O R 4150 4250 50
+F9 "SERVO5" O R 4150 4350 50
+F10 "SERVO6" O R 4150 4450 50
+F11 "SERVO7" O R 4150 4550 50
+F12 "SERVO8" O R 4150 4650 50
+F13 "SERVO9" O R 4150 4750 50
+F14 "SERVO10" O R 4150 4850 50
+F15 "SERVO11" O R 4150 4950 50
+F16 "SERVO12" O R 4150 5050 50
+F17 "SERVO13" O R 4150 5150 50
+F18 "SERVO14" O R 4150 5250 50
+F19 "SERVO15" O R 4150 5350 50
+F20 "SERVO16" O R 4150 5450 50
+F21 "SERVO17" O R 4150 5550 50
+F22 "SERVO18" O R 4150 5650 50
+F23 "SERVO19" O R 4150 5750 50
+$EndSheet
+Text Label 4150 3850 0    50   ~ 0
+SERVO0
+Text Label 4150 3950 0    50   ~ 0
+SERVO1
+Text Label 4150 4050 0    50   ~ 0
+SERVO2
+Text Label 4150 4150 0    50   ~ 0
+SERVO3
+Text Label 4150 4250 0    50   ~ 0
+SERVO4
+Text Label 4150 4350 0    50   ~ 0
+SERVO5
+Text Label 4150 4450 0    50   ~ 0
+SERVO6
+Text Label 4150 4550 0    50   ~ 0
+SERVO7
+Text Label 4150 4650 0    50   ~ 0
+SERVO8
+Text Label 4150 4750 0    50   ~ 0
+SERVO9
+Text Label 4150 4850 0    50   ~ 0
+SERVO10
+Text Label 4150 4950 0    50   ~ 0
+SERVO11
+Text Label 4150 5050 0    50   ~ 0
+SERVO12
+Text Label 4150 5150 0    50   ~ 0
+SERVO13
+Text Label 4150 5250 0    50   ~ 0
+SERVO14
+Text Label 4150 5350 0    50   ~ 0
+SERVO15
+Text Label 4150 5450 0    50   ~ 0
+SERVO16
+Text Label 4150 5550 0    50   ~ 0
+SERVO17
+Text Label 4150 5650 0    50   ~ 0
+SERVO18
+Text Label 4150 5750 0    50   ~ 0
+SERVO19
+Wire Wire Line
+	1850 1950 1350 1950
+Text Label 7250 3350 2    50   ~ 0
+NRST
+Text Label 7250 3450 2    50   ~ 0
+TX1
+Text Label 7250 3550 2    50   ~ 0
+RX1
+Text Label 1850 2250 2    50   ~ 0
+TX1
+Text Label 1850 1350 2    50   ~ 0
+RX1
+Text Label 1850 1150 2    50   ~ 0
+NRST
+Text Label 9800 1200 2    50   ~ 0
+SAFETYSDA
+Text Label 9800 1100 2    50   ~ 0
+SAFETYSCL
+Text Label 7250 3950 2    50   ~ 0
+SAFETYSDA
+Text Label 7250 3850 2    50   ~ 0
+SAFETYSCL
+Text Label 7250 3650 2    50   ~ 0
+TALKALLOWED
+Text Label 7250 3750 2    50   ~ 0
+TALKING
+Text Label 1850 1250 2    50   ~ 0
+TALKALLOWED
+Text Label 10950 2650 0    50   ~ 0
+SDA
+Text Label 9750 4200 2    50   ~ 0
+SERVO16
+Text Label 9750 4300 2    50   ~ 0
+SERVO17
+Text Label 9750 4400 2    50   ~ 0
+SERVO18
+Text Label 9750 4500 2    50   ~ 0
+SERVO19
 $EndSCHEMATC

Commit message: This rev removes the safety micro and instead uses the dji battery
Parts:
- removed J9: Conn_01x02_Male, XT30PB:XT30PB, symbol Connector:Conn_01x02_Male
- added C17: 0.1uF, Capacitor_SMD:C_0402_1005Metric, symbol Device:C
- added J18: Micro_SD_Card, Connector_Card:microSD_HC_Wuerth_693072010801, symbol Connector:Micro_SD_Card
- added J9: Conn_01x10_Female, Connector_JST:JST_EH_B10B-EH-A_1x10_P2.50mm_Vertical, symbol Connector:Conn_01x10_Female
- added R2, R22: 10K, Resistor_SMD:R_0402_1005Metric, symbol Device:R
- added R23: 8.2K, Resistor_SMD:R_0402_1005Metric, symbol Device:R
- added R3: 2.4K, Resistor_SMD:R_0402_1005Metric, symbol Device:R
- added U2: PCA9685BS, Package_DFN_QFN:QFN-28-1EP_6x6mm_P0.65mm_EP4.25x4.25mm, symbol Driver_LED:PCA9685BS
Connections:
- net labels added: +3.3V, BATT_VOLTAGE, EN_SERVO_DRIVER, IO12, IO13, IO14, IO15, IO2, IO4, MEASURED_6V, MEASURED_FUSE1, MEASURED_FUSE2, MEASURED_FUSE3, MEASURED_FUSE4
- net labels removed: 3.3VEN, CC1, CC2, NRST, RX1, SAFETYSCL, SAFETYSDA, SERVO16, SERVO17, SERVO18, SERVO19, TALKALLOWED, TALKING, TX1
- wire segments 8 -> 20
- no-connect marks 0 -> 2
Other:
- moved on the sheet: TP1, TP2, TP3

Commit message: rev, pendingorder
Parts:
- added D9: LED, LED_SMD:LED_0603_1608Metric, symbol Device:LED
- added F5: Fuse, 01550900M:0154.250DR, symbol Device:Fuse
- added J20: Qwiic connector, Connector_JST:JST_SH_SM04B-SRSS-TB_1x04-1MP_P1.00mm_Horizontal, symbol Connector:Conn_01x04_Female
- added J21, J22, J23, J24: Conn_01x03_Male, Connector_PinHeader_2.54mm:PinHeader_1x03_P2.54mm_Vertical, symbol Connector:Conn_01x03_Male
- added R17: 10K, Resistor_SMD:R_0402_1005Metric, symbol Device:R
- added R24: 8.2K, Resistor_SMD:R_0402_1005Metric, symbol Device:R
- added R39: 20K, Resistor_SMD:R_0402_1005Metric, symbol Device:R
- J18: footprint Connector_Card:microSD_HC_Wuerth_693072010801 -> Connector_Card:microSD_HC_Molex_104031-0811
- J9: value Conn_01x10_Female -> DJI Battery Connector
- TP1: value TestPoint -> Check for life
- TP2: value TestPoint -> SDA
- TP3: value TestPoint -> SCL
Connections:
- net +3V3: now also J20.2 (Pin_2)
- net +6V: now also F5.2
- net GND: now also D9.1 (K), J20.1 (Pin_1), J21.3 (Pin_3), J22.3 (Pin_3), J23.3 (Pin_3), J24.3 (Pin_3), R24.2
- net SCL: now also J20.4 (Pin_4)
- net SDA: now also J20.3 (Pin_3)
- new net: D9.2 (A), R39.2
- new net AD_6V: F5.1, J21.2 (Pin_2), J22.2 (Pin_2), J23.2 (Pin_2), J24.2 (Pin_2), R17.1, R39.1
- new net AD_SERVO_1: J21.1 (Pin_1)
- new net AD_SERVO_2: J23.1 (Pin_1)
- new net AD_SERVO_3: J22.1 (Pin_1)
- new net AD_SERVO_4: J24.1 (Pin_1)
- new net MEASURED_FUSE5: R17.2, R24.1
Other:
- note added: "Additional Servos"
- note added: "DJI Battery"
- note added: "ESP32, USB & USB -> Serial"
- note added: "IMU"
- note added: "Mounting Holes"
- note added: "Power Monitoring"
- note added: "Power Regulators"
- note added: "QWICC"
- note added: "SD Card"
- note added: "Servo Breakouts"
- note added: "Servo Expander"
- note added: "Test Points"
- moved on the sheet: C17, D2, H1, H2, H3, H4, J18, J9, R2, R22, R23, R3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

Commit message: g
Parts:
- added J25: Conn_01x02_Female, RC-Battery-Connectors:XT-60_male, symbol Connector:Conn_01x02_Female
- added J26: Conn_01x02_Female, RC-Battery-Connectors:XT-60_female, symbol Connector:Conn_01x02_Female
- renumbered C17 to C1, D9 to D3, F5 to F1, J9 to J1, J20 to J2, J21 to J3, J22 to J4, J23 to J5, J24 to J6, J18 to J7, R22 to R4, R23 to R5, R17 to R7, R24 to R8, R39 to R9, U2 to U1
Connections:
- net +BATT: now also J25.2 (Pin_2); no longer J1.10 (Pin_10), J1.7 (Pin_7), J1.8 (Pin_8), J1.9 (Pin_9)
- net GND: now also J25.1 (Pin_1), J26.1 (Pin_1)
- new net: J1.10 (Pin_10), J1.7 (Pin_7), J1.8 (Pin_8), J1.9 (Pin_9), J26.2 (Pin_2)
Other:
- note added: "Battery"
- note added: "DJI to XT-30"
- note removed: "DJI Battery"
- moved on the sheet: D3, F1, J1, R9
