File: MainBoard.sch (KiCad schematic (older format))
At the start: 31 parts, among them J1 DJI Battery Connector, J2 Qwiic connector, J25 Conn_01x02_Female, J26 Conn_01x02_Female, J3 Conn_01x03_Male, J4 Conn_01x03_Male, J5 Conn_01x03_Male, J6 Conn_01x03_Male, J7 Micro_SD_Card, U1 PCA9685BS

Commit message: rev ordered
Parts:
- removed J1: DJI Battery Connector, Connector_JST:JST_EH_B10B-EH-A_1x10_P2.50mm_Vertical, symbol Connector:Conn_01x10_Female
- removed J26: Conn_01x02_Female, RC-Battery-Connectors:XT-60_female, symbol Connector:Conn_01x02_Female
- added R44, R45, R46: 10K, Resistor_SMD:R_0402_1005Metric, symbol Device:R
- added TP12: SDA, TestPoint:TestPoint_Pad_D1.5mm, symbol Connector:TestPoint
- added TP13: SCL, TestPoint:TestPoint_Pad_D1.5mm, symbol Connector:TestPoint
Connections:
- net labels added: SCL_1, SDA_1
- wire segments 25 -> 14
- no-connect marks 2 -> 0
Other:
- note removed: "DJI to XT-30"
- moved on the sheet: TP2, TP3

Commit message: Final order version with all bom files
Parts:
- added J1: Qwiic connector, Connector_JST:JST_SH_SM04B-SRSS-TB_1x04-1MP_P1.00mm_Horizontal, symbol Connector:Conn_01x04_Female
- added R14: 10K, Resistor_SMD:R_0402_1005Metric, symbol Device:R
Connections:
- net +3V3: now also J1.2 (Pin_2)
- net EN_SERVO_DRIVER: now also R14.1
- net GND: now also J1.1 (Pin_1), R14.2
- net SCL_1: now also J1.3 (Pin_3)
- net SDA_1: now also J1.4 (Pin_4)
Changed lines of the file:
@@
 $EndComp
 $Sheet
-S 10150 4150 800  1700
+S 5950 5750 800  1700
 U 5DD5998B
 F0 "Servos" 50
 F1 "Servos.sch" 50
-F2 "SERVO1" I L 10150 4250 50
-F3 "SERVO2" I L 10150 4350 50
-F4 "SERVO3" I L 10150 4450 50
-F5 "SERVO4" I L 10150 4550 50
-F6 "SERVO5" I L 10150 4650 50
-F7 "SERVO6" I L 10150 4750 50
-F8 "SERVO7" I L 10150 4850 50
-F9 "SERVO8" I L 10150 4950 50
-F10 "SERVO9" I L 10150 5050 50
-F11 "SERVO10" I L 10150 5150 50
-F12 "SERVO11" I L 10150 5250 50
-F13 "SERVO12" I L 10150 5350 50
-F14 "SERVO13" I L 10150 5450 50
-F15 "SERVO14" I L 10150 5550 50
-F16 "SERVO15" I L 10150 5650 50
-F17 "SERVO16" I L 10150 5750 50
+F2 "SERVO1" I L 5950 5850 50
+F3 "SERVO2" I L 5950 5950 50
+F4 "SERVO3" I L 5950 6050 50
+F5 "SERVO4" I L 5950 6150 50
+F6 "SERVO5" I L 5950 6250 50
+F7 "SERVO6" I L 5950 6350 50
+F8 "SERVO7" I L 5950 6450 50
+F9 "SERVO8" I L 5950 6550 50
+F10 "SERVO9" I L 5950 6650 50
+F11 "SERVO10" I L 5950 6750 50
+F12 "SERVO11" I L 5950 6850 50
+F13 "SERVO12" I L 5950 6950 50
+F14 "SERVO13" I L 5950 7050 50
+F15 "SERVO14" I L 5950 7150 50
+F16 "SERVO15" I L 5950 7250 50
+F17 "SERVO16" I L 5950 7350 50
 $EndSheet
 $Sheet
@@
 Text Label 5300 1600 2    50   ~ 0
 SDA_1
-Text Label 10150 5750 2    50   ~ 0
+Text Label 5950 7350 2    50   ~ 0
 SERVO15
-Text Label 10150 5650 2    50   ~ 0
+Text Label 5950 7250 2    50   ~ 0
 SERVO14
-Text Label 10150 5550 2    50   ~ 0
+Text Label 5950 7150 2    50   ~ 0
 SERVO13
-Text Label 10150 5450 2    50   ~ 0
+Text Label 5950 7050 2    50   ~ 0
 SERVO12
-Text Label 10150 5350 2    50   ~ 0
+Text Label 5950 6950 2    50   ~ 0
 SERVO11
-Text Label 10150 5250 2    50   ~ 0
+Text Label 5950 6850 2    50   ~ 0
 SERVO10
-Text Label 10150 5150 2    50   ~ 0
+Text Label 5950 6750 2    50   ~ 0
 SERVO9
-Text Label 10150 5050 2    50   ~ 0
+Text Label 5950 6650 2    50   ~ 0
 SERVO8
-Text Label 10150 4950 2    50   ~ 0
+Text Label 5950 6550 2    50   ~ 0
 SERVO7
-Text Label 10150 4850 2    50   ~ 0
+Text Label 5950 6450 2    50   ~ 0
 SERVO6
-Text Label 10150 4750 2    50   ~ 0
+Text Label 5950 6350 2    50   ~ 0
 SERVO5
-Text Label 10150 4650 2    50   ~ 0
+Text Label 5950 6250 2    50   ~ 0
 SERVO4
-Text Label 10150 4550 2    50   ~ 0
+Text Label 5950 6150 2    50   ~ 0
 SERVO3
-Text Label 10150 4450 2    50   ~ 0
+Text Label 5950 6050 2    50   ~ 0
 SERVO2
-Text Label 10150 4350 2    50   ~ 0
+Text Label 5950 5950 2    50   ~ 0
 SERVO1
-Text Label 10150 4250 2    50   ~ 0
+Text Label 5950 5850 2    50   ~ 0
 SERVO0
 Text Label 6700 3000 0    50   ~ 0
@@
 Power Regulators
 Wire Notes Line
-	5350 6850 5350 5600
-Wire Notes Line
 	450  6850 5350 6850
 Text Notes 3450 6850 0    118  ~ 24
 Power Monitoring
 Wire Notes Line
-	9550 4000 9550 6250
-Wire Notes Line
-	9550 6250 11250 6250
-Text Notes 9650 6200 0    118  ~ 24
+	5350 7850 7050 7850
+Text Notes 5450 7800 0    118  ~ 24
 Servo Breakouts
 Text Notes 700  5150 0    118  ~ 24
@@
 SDA_1
 Wire Notes Line
+	7400 4000 7400 450
+Wire Notes Line
+	6950 5600 3200 5600
+$Comp
+L Device:R R?
+U 1 1 5FE2B7C0
+P 5300 1950
+AR Path="/5FE2B7C0" Ref="R?"  Part="1"
+AR Path="/5DAA9390/5FE2B7C0" Ref="R14"  Part="1"
+AR Path="/5DAA9390/5DAAB924/5FE2B7C0" Ref="R?"  Part="1"
+AR Path="/5DAA9E7A/5DB7E2D8/5FE2B7C0" Ref="R?"  Part="1"
+AR Path="/5FFBF360/5FE2B7C0" Ref="R?"  Part="1"
+AR Path="/5DAAB924/5FE2B7C0" Ref="R?"  Part="1"
+F 0 "R14" V 5093 1950 50  0000 C CNN
+F 1 "10K" V 5184 1950 50  0000 C CNN
+F 2 "Resistor_SMD:R_0402_1005Metric" V 5230 1950 50  0001 C CNN
+F 3 "~" H 5300 1950 50  0001 C CNN
+	1    5300 1950
+	1    0    0    -1
+$EndComp
+$Comp
+L power:GND #PWR0208
+U 1 1 5FE2D2D9
+P 5300 2100
+F 0 "#PWR0208" H 5300 1850 50  0001 C CNN
+F 1 "GND" H 5305 1927 50  0000 C CNN
+F 2 "" H 5300 2100 50  0001 C CNN
+F 3 "" H 5300 2100 50  0001 C CNN
+	1    5300 2100
+	1    0    0    -1
+$EndComp
+$Comp
+L power:GND #PWR0214
+U 1 1 5FFFCBC7
+P 1300 7550
+F 0 "#PWR0214" H 1300 7300 50  0001 C CNN
+F 1 "GND" H 1305 7377 50  0000 C CNN
+F 2 "" H 1300 7550 50  0001 C CNN
+F 3 "" H 1300 7550 50  0001 C CNN
+	1    1300 7550
+	1    0    0    -1
+$EndComp
+Wire Wire Line
+	1300 7300 1300 7550
+$Comp
+L Connector:Conn_01x04_Female J1
+U 1 1 5FFFCBCE
+P 1400 7100
+F 0 "J1" V 1550 7150 50  0000 R CNN
+F 1 "Qwiic connector" V 1450 7400 50  0000 R CNN
+F 2 "Connector_JST:JST_SH_SM04B-SRSS-TB_1x04-1MP_P1.00mm_Horizontal" H 1400 7100 50  0001 C CNN
+F 3 "~" H 1400 7100 50  0001 C CNN
+	1    1400 7100
+	0    -1   -1   0
+$EndComp
+$Comp
+L power:+3.3V #PWR0215
+U 1 1 5FFFCBD4
+P 1400 7300
+F 0 "#PWR0215" H 1400 7150 50  0001 C CNN
+F 1 "+3.3V" H 1415 7473 50  0000 C CNN
+F 2 "" H 1400 7300 50  0001 C CNN
+F 3 "" H 1400 7300 50  0001 C CNN
+	1    1400 7300
+	-1   0    0    1
+$EndComp
+Text Label 1500 7300 3    50   ~ 0
+SCL_1
+Text Label 1600 7300 3    50   ~ 0
+SDA_1
+Wire Notes Line
+	5350 5600 5350 7850
+Wire Notes Line
 	500  4000 11250 4000
-Wire Notes Line
-	7400 4000 7400 450
-Wire Notes Line
-	6950 5600 3200 5600
 $EndSCHEMATC
