File: BNO055.sch (KiCad schematic (older format))
At the start: 6 parts, among them U1 BNO055, Y1 32.768kHz

Commit message: This rev removes the safety micro and instead uses the dji battery
Parts:
- U1: symbol Sensor_Motion:BNO055 -> SmallKat-v2-rescue:BNO055-Sensor_Motion-SmallKat-v2-rescue
Changed lines of the file:
@@
 $Descr A4 11693 8268
 encoding utf-8
-Sheet 4 12
+Sheet 4 7
 Title ""
 Date ""
@@
 $EndDescr
 $Comp
-L Sensor_Motion:BNO055 U?
+L SmallKat-v2-rescue:BNO055-Sensor_Motion-SmallKat-v2-rescue U?
 U 1 1 5DAC5A25
 P 5350 3550

Commit message: batt connector and all in the right place. has not been ordered, waiting for prev rev to be tested first
Parts:
- U1: symbol SmallKat-v2-rescue:BNO055-Sensor_Motion-SmallKat-v2-rescue -> SmallKat-v2-rescue:BNO055-Sensor_Motion-SmallKat-v2-rescue-SmallKat-v2-rescue
Changed lines of the file:
@@
 $EndDescr
 $Comp
-L SmallKat-v2-rescue:BNO055-Sensor_Motion-SmallKat-v2-rescue U?
+L SmallKat-v2-rescue:BNO055-Sensor_Motion-SmallKat-v2-rescue-SmallKat-v2-rescue U?
 U 1 1 5DAC5A25
 P 5350 3550

Commit message: rev, pendingorder
Parts:
- U1: symbol SmallKat-v2-rescue:BNO055-Sensor_Motion-SmallKat-v2-rescue-SmallKat-v2-rescue -> SmallKat-v2-rescue:BNO055-Sensor_Motion-SmallKat-v2-rescue-SmallKat-v2-rescue-SmallKat-v2-rescue-SmallKat-v2-rescue-Sma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
Changed lines of the file:
@@
 $EndDescr
 $Comp
-L SmallKat-v2-rescue:BNO055-Sensor_Motion-SmallKat-v2-rescue-SmallKat-v2-rescue U?
+L SmallKat-v2-rescue:BNO055-Sensor_Motion-SmallKat-v2-rescue-SmallKat-v2-rescue-SmallKat-v2-rescue-SmallKat-v2-rescue-SmallKat-v2-rescue-SmallKat-v2-rescue U?
 U 1 1 5DAC5A25
 P 5350 3550
 AR Path="/5DAC5A25" Ref="U?"  Part="1"
 AR Path="/5DAA9390/5DAC4399/5DAC5A25" Ref="U1"  Part="1"
-F 0 "U1" H 5350 3550 50  0000 C CNN
+F 0 "U?" H 5350 3550 50  0000 C CNN
 F 1 "BNO055" H 5350 3900 50  0000 C CNN
 F 2 "Package_LGA:LGA-28_5.2x3.8mm_P0.5mm" H 5600 2900 50  0001 L CNN
@@
 AR Path="/5DAC5A2D" Ref="#PWR?"  Part="1"
 AR Path="/5DAA9390/5DAC4399/5DAC5A2D" Ref="#PWR0142"  Part="1"
-F 0 "#PWR0142" H 4750 3700 50  0001 C CNN
+F 0 "#PWR?" H 4750 3700 50  0001 C CNN
 F 1 "GND" V 4755 3822 50  0000 R CNN
 F 2 "" H 4750 3950 50  0001 C CNN
@@
 AR Path="/5DAC5A33" Ref="R?"  Part="1"
 AR Path="/5DAA9390/5DAC4399/5DAC5A33" Ref="R11"  Part="1"
-F 0 "R11" V 4700 4050 50  0000 C CNN
+F 0 "R?" V 4700 4050 50  0000 C CNN
 F 1 "10K" V 4700 4150 50  0000 C CNN
 F 2 "Resistor_SMD:R_0402_1005Metric" V 4530 4050 50  0001 C CNN
@@
 AR Path="/5DAC5A39" Ref="#PWR?"  Part="1"
 AR Path="/5DAA9390/5DAC4399/5DAC5A39" Ref="#PWR0143"  Part="1"
-F 0 "#PWR0143" H 4450 3800 50  0001 C CNN
+F 0 "#PWR?" H 4450 3800 50  0001 C CNN
 F 1 "GND" H 4455 3877 50  0000 C CNN
 F 2 "" H 4450 4050 50  0001 C CNN
@@
 AR Path="/5DAC5A41" Ref="Y?"  Part="1"
 AR Path="/5DAA9390/5DAC4399/5DAC5A41" Ref="Y1"  Part="1"
-F 0 "Y1" H 6150 3000 50  0000 L CNN
+F 0 "Y?" H 6150 3000 50  0000 L CNN
 F 1 "32.768kHz" H 6050 3100 50  0000 L CNN
 F 2 "Crystal:Crystal_SMD_3215-2Pin_3.2x1.5mm" H 6200 3250 50  0001 C CNN
@@
 AR Path="/5DAC5A4B" Ref="C?"  Part="1"
 AR Path="/5DAA9390/5DAC4399/5DAC5A4B" Ref="C9"  Part="1"
-F 0 "C9" V 6200 3400 50  0000 C CNN
+F 0 "C?" V 6200 3400 50  0000 C CNN
 F 1 "10pF" V 6500 3400 50  0000 C CNN
 F 2 "Capacitor_SMD:C_0402_1005Metric" H 6388 3250 50  0001 C CNN
@@
 AR Path="/5DAC5A52" Ref="C?"  Part="1"
 AR Path="/5DAA9390/5DAC4399/5DAC5A52" Ref="C8"  Part="1"
-F 0 "C8" V 6098 3100 50  0000 C CNN
+F 0 "C?" V 6098 3100 50  0000 C CNN
 F 1 "10pF" V 6189 3100 50  0000 C CNN
 F 2 "Capacitor_SMD:C_0402_1005Metric" H 6388 2950 50  0001 C CNN
@@
 AR Path="/5DAC5A5A" Ref="#PWR?"  Part="1"
 AR Path="/5DAA9390/5DAC4399/5DAC5A5A" Ref="#PWR0144"  Part="1"
-F 0 "#PWR0144" H 6500 3000 50  0001 C CNN
+F 0 "#PWR?" H 6500 3000 50  0001 C CNN
 F 1 "GND" V 6505 3122 50  0000 R CNN
 F 2 "" H 6500 3250 50  0001 C CNN
@@
 AR Path="/5DAC5A62" Ref="#PWR?"  Part="1"
 AR Path="/5DAA9390/5DAC4399/5DAC5A62" Ref="#PWR0145"  Part="1"
-F 0 "#PWR0145" H 5250 4000 50  0001 C CNN
+F 0 "#PWR?" H 5250 4000 50  0001 C CNN
 F 1 "GND" H 5255 4077 50  0000 C CNN
 F 2 "" H 5250 4250 50  0001 C CNN
@@
 AR Path="/5DAC5A68" Ref="#PWR?"  Part="1"
 AR Path="/5DAA9390/5DAC4399/5DAC5A68" Ref="#PWR0146"  Part="1"
-F 0 "#PWR0146" H 5450 4000 50  0001 C CNN
+F 0 "#PWR?" H 5450 4000 50  0001 C CNN
 F 1 "GND" H 5455 4077 50  0000 C CNN
 F 2 "" H 5450 4250 50  0001 C CNN
@@
 AR Path="/5DAC5A6E" Ref="#PWR?"  Part="1"
 AR Path="/5DAA9390/5DAC4399/5DAC5A6E" Ref="#PWR0147"  Part="1"
-F 0 "#PWR0147" H 5250 2700 50  0001 C CNN
+F 0 "#PWR?" H 5250 2700 50  0001 C CNN
 F 1 "+3.3V" H 5265 3023 50  0000 C CNN
 F 2 "" H 5250 2850 50  0001 C CNN
@@
 AR Path="/5DAC5A74" Ref="#PWR?"  Part="1"
 AR Path="/5DAA9390/5DAC4399/5DAC5A74" Ref="#PWR0148"  Part="1"
-F 0 "#PWR0148" H 4750 3300 50  0001 C CNN
+F 0 "#PWR?" H 4750 3300 50  0001 C CNN
 F 1 "+3.3V" H 4765 3623 50  0000 C CNN
 F 2 "" H 4750 3450 50  0001 C CNN
@@
 AR Path="/5DAC5A7A" Ref="#PWR?"  Part="1"
 AR Path="/5DAA9390/5DAC4399/5DAC5A7A" Ref="#PWR0149"  Part="1"
-F 0 "#PWR0149" H 5950 3600 50  0001 C CNN
+F 0 "#PWR?" H 5950 3600 50  0001 C CNN
 F 1 "GND" V 5950 3700 50  0000 R CNN
 F 2 "" H 5950 3850 50  0001 C CNN
@@
 AR Path="/5DAC5A80" Ref="#PWR?"  Part="1"
 AR Path="/5DAA9390/5DAC4399/5DAC5A80" Ref="#PWR0150"  Part="1"
-F 0 "#PWR0150" H 5950 3700 50  0001 C CNN
+F 0 "#PWR?" H 5950 3700 50  0001 C CNN
 F 1 "GND" V 5955 3822 50  0000 R CNN
 F 2 "" H 5950 3950 50  0001 C CNN
@@
 AR Path="/5DAC5A86" Ref="C?"  Part="1"
 AR Path="/5DAA9390/5DAC4399/5DAC5A86" Ref="C7"  Part="1"
-F 0 "C7" V 6250 3950 50  0000 C CNN
+F 0 "C?" V 6250 3950 50  0000 C CNN
 F 1 "0.1uF" V 6250 4050 50  0000 C CNN
 F 2 "Capacitor_SMD:C_0402_1005Metric" H 6138 3900 50  0001 C CNN
@@
 AR Path="/5DAC5A8C" Ref="#PWR?"  Part="1"
 AR Path="/5DAA9390/5DAC4399/5DAC5A8C" Ref="#PWR0151"  Part="1"
-F 0 "#PWR0151" H 6250 3800 50  0001 C CNN
+F 0 "#PWR?" H 6250 3800 50  0001 C CNN
 F 1 "GND" H 6255 3877 50  0000 C CNN
 F 2 "" H 6250 4050 50  0001 C CNN
@@
 AR Path="/5DAC5A92" Ref="#PWR?"  Part="1"
 AR Path="/5DAA9390/5DAC4399/5DAC5A92" Ref="#PWR0152"  Part="1"
-F 0 "#PWR0152" H 5450 2700 50  0001 C CNN
+F 0 "#PWR?" H 5450 2700 50  0001 C CNN
 F 1 "+3.3V" H 5465 3023 50  0000 C CNN
 F 2 "" H 5450 2850 50  0001 C CNN

Commit message: g
Parts:
- U2: renamed from U1; symbol SmallKat-v2-rescue:BNO055-Sensor_Motion-SmallKat-v2-rescue-SmallKat-v2-rescue-SmallKat-v2-rescue-SmallKat-v2-rescue-SmallKat-v2-rescue-SmallKat-v2-rescue -> SmallKat-v2-rescue:BNO055-Sensor_Motion-SmallKat-v2-rescue-SmallKat-v2-rescue-SmallKat-v2-rescue-SmallKat-v2-rescue-SmallKat-v2-rescue-SmallKat-v2-rescue-SmallKat-v2-rescue-SmallKat-v2-rescue
- renumbered C7 to C14, C8 to C15, C9 to C16, R11 to R17
Changed lines of the file:
@@
 $Descr A4 11693 8268
 encoding utf-8
-Sheet 4 7
+Sheet 3 7
 Title ""
 Date ""
@@
 $EndDescr
 $Comp
-L SmallKat-v2-rescue:BNO055-Sensor_Motion-SmallKat-v2-rescue-SmallKat-v2-rescue-SmallKat-v2-rescue-SmallKat-v2-rescue-SmallKat-v2-rescue-SmallKat-v2-rescue U?
+L SmallKat-v2-rescue:BNO055-Sensor_Motion-SmallKat-v2-rescue-SmallKat-v2-rescue-SmallKat-v2-rescue-SmallKat-v2-rescue-SmallKat-v2-rescue-SmallKat-v2-rescue-SmallKat-v2-rescue-SmallKat-v2-rescue U?
 U 1 1 5DAC5A25
 P 5350 3550
 AR Path="/5DAC5A25" Ref="U?"  Part="1"
-AR Path="/5DAA9390/5DAC4399/5DAC5A25" Ref="U1"  Part="1"
-F 0 "U?" H 5350 3550 50  0000 C CNN
+AR Path="/5DAA9390/5DAC4399/5DAC5A25" Ref="U2"  Part="1"
+AR Path="/5FFBF36C/5DAC5A25" Ref="U?"  Part="1"
+AR Path="/5DAC4399/5DAC5A25" Ref="U2"  Part="1"
+F 0 "U2" H 5350 3550 50  0000 C CNN
 F 1 "BNO055" H 5350 3900 50  0000 C CNN
 F 2 "Package_LGA:LGA-28_5.2x3.8mm_P0.5mm" H 5600 2900 50  0001 L CNN
@@
 P 4750 3950
 AR Path="/5DAC5A2D" Ref="#PWR?"  Part="1"
-AR Path="/5DAA9390/5DAC4399/5DAC5A2D" Ref="#PWR0142"  Part="1"
-F 0 "#PWR?" H 4750 3700 50  0001 C CNN
+AR Path="/5DAA9390/5DAC4399/5DAC5A2D" Ref="#PWR0127"  Part="1"
+AR Path="/5FFBF36C/5DAC5A2D" Ref="#PWR?"  Part="1"
+AR Path="/5DAC4399/5DAC5A2D" Ref="#PWR054"  Part="1"
+F 0 "#PWR0127" H 4750 3700 50  0001 C CNN
 F 1 "GND" V 4755 3822 50  0000 R CNN
 F 2 "" H 4750 3950 50  0001 C CNN
@@
 P 4600 4050
 AR Path="/5DAC5A33" Ref="R?"  Part="1"
-AR Path="/5DAA9390/5DAC4399/5DAC5A33" Ref="R11"  Part="1"
-F 0 "R?" V 4700 4050 50  0000 C CNN
+AR Path="/5DAA9390/5DAC4399/5DAC5A33" Ref="R17"  Part="1"
+AR Path="/5FFBF36C/5DAC5A33" Ref="R?"  Part="1"
+AR Path="/5DAC4399/5DAC5A33" Ref="R17"  Part="1"
+F 0 "R17" V 4700 4050 50  0000 C CNN
 F 1 "10K" V 4700 4150 50  0000 C CNN
 F 2 "Resistor_SMD:R_0402_1005Metric" V 4530 4050 50  0001 C CNN
@@
 P 4450 4050
 AR Path="/5DAC5A39" Ref="#PWR?"  Part="1"
-AR Path="/5DAA9390/5DAC4399/5DAC5A39" Ref="#PWR0143"  Part="1"
-F 0 "#PWR?" H 4450 3800 50  0001 C CNN
+AR Path="/5DAA9390/5DAC4399/5DAC5A39" Ref="#PWR0128"  Part="1"
+AR Path="/5FFBF36C/5DAC5A39" Ref="#PWR?"  Part="1"
+AR Path="/5DAC4399/5DAC5A39" Ref="#PWR052"  Part="1"
+F 0 "#PWR0128" H 4450 3800 50  0001 C CNN
 F 1 "GND" H 4455 3877 50  0000 C CNN
 F 2 "" H 4450 4050 50  0001 C CNN
@@
 AR Path="/5DAC5A41" Ref="Y?"  Part="1"
 AR Path="/5DAA9390/5DAC4399/5DAC5A41" Ref="Y1"  Part="1"
-F 0 "Y?" H 6150 3000 50  0000 L CNN
+AR Path="/5FFBF36C/5DAC5A41" Ref="Y?"  Part="1"
+AR Path="/5DAC4399/5DAC5A41" Ref="Y1"  Part="1"
+F 0 "Y1" H 6150 3000 50  0000 L CNN
 F 1 "32.768kHz" H 6050 3100 50  0000 L CNN
 F 2 "Crystal:Crystal_SMD_3215-2Pin_3.2x1.5mm" H 6200 3250 50  0001 C CNN
@@
 P 6350 3400
 AR Path="/5DAC5A4B" Ref="C?"  Part="1"
-AR Path="/5DAA9390/5DAC4399/5DAC5A4B" Ref="C9"  Part="1"
-F 0 "C?" V 6200 3400 50  0000 C CNN
+AR Path="/5DAA9390/5DAC4399/5DAC5A4B" Ref="C16"  Part="1"
+AR Path="/5FFBF36C/5DAC5A4B" Ref="C?"  Part="1"
+AR Path="/5DAC4399/5DAC5A4B" Ref="C16"  Part="1"
+F 0 "C16" V 6200 3400 50  0000 C CNN
 F 1 "10pF" V 6500 3400 50  0000 C CNN
 F 2 "Capacitor_SMD:C_0402_1005Metric" H 6388 3250 50  0001 C CNN
@@
 P 6350 3100
 AR Path="/5DAC5A52" Ref="C?"  Part="1"
-AR Path="/5DAA9390/5DAC4399/5DAC5A52" Ref="C8"  Part="1"
-F 0 "C?" V 6098 3100 50  0000 C CNN
+AR Path="/5DAA9390/5DAC4399/5DAC5A52" Ref="C15"  Part="1"
+AR Path="/5FFBF36C/5DAC5A52" Ref="C?"  Part="1"
+AR Path="/5DAC4399/5DAC5A52" Ref="C15"  Part="1"
+F 0 "C15" V 6098 3100 50  0000 C CNN
 F 1 "10pF" V 6189 3100 50  0000 C CNN
 F 2 "Capacitor_SMD:C_0402_1005Metric" H 6388 2950 50  0001 C CNN
@@
 P 6500 3250
 AR Path="/5DAC5A5A" Ref="#PWR?"  Part="1"
-AR Path="/5DAA9390/5DAC4399/5DAC5A5A" Ref="#PWR0144"  Part="1"
-F 0 "#PWR?" H 6500 3000 50  0001 C CNN
+AR Path="/5DAA9390/5DAC4399/5DAC5A5A" Ref="#PWR0129"  Part="1"
+AR Path="/5FFBF36C/5DAC5A5A" Ref="#PWR?"  Part="1"
+AR Path="/5DAC4399/5DAC5A5A" Ref="#PWR062"  Part="1"
+F 0 "#PWR0129" H 6500 3000 50  0001 C CNN
 F 1 "GND" V 6505 3122 50  0000 R CNN
 F 2 "" H 6500 3250 50  0001 C CNN
@@
 P 5250 4250
 AR Path="/5DAC5A62" Ref="#PWR?"  Part="1"
-AR Path="/5DAA9390/5DAC4399/5DAC5A62" Ref="#PWR0145"  Part="1"
-F 0 "#PWR?" H 5250 4000 50  0001 C CNN
+AR Path="/5DAA9390/5DAC4399/5DAC5A62" Ref="#PWR0130"  Part="1"
+AR Path="/5FFBF36C/5DAC5A62" Ref="#PWR?"  Part="1"
+AR Path="/5DAC4399/5DAC5A62" Ref="#PWR056"  Part="1"
+F 0 "#PWR0130" H 5250 4000 50  0001 C CNN
 F 1 "GND" H 5255 4077 50  0000 C CNN
 F 2 "" H 5250 4250 50  0001 C CNN
@@
 P 5450 4250
 AR Path="/5DAC5A68" Ref="#PWR?"  Part="1"
-AR Path="/5DAA9390/5DAC4399/5DAC5A68" Ref="#PWR0146"  Part="1"
-F 0 "#PWR?" H 5450 4000 50  0001 C CNN
+AR Path="/5DAA9390/5DAC4399/5DAC5A68" Ref="#PWR0131"  Part="1"
+AR Path="/5FFBF36C/5DAC5A68" Ref="#PWR?"  Part="1"
+AR Path="/5DAC4399/5DAC5A68" Ref="#PWR058"  Part="1"
+F 0 "#PWR0131" H 5450 4000 50  0001 C CNN
 F 1 "GND" H 5455 4077 50  0000 C CNN
 F 2 "" H 5450 4250 50  0001 C CNN
@@
 P 5250 2850
 AR Path="/5DAC5A6E" Ref="#PWR?"  Part="1"
-AR Path="/5DAA9390/5DAC4399/5DAC5A6E" Ref="#PWR0147"  Part="1"
-F 0 "#PWR?" H 5250 2700 50  0001 C CNN
+AR Path="/5DAA9390/5DAC4399/5DAC5A6E" Ref="#PWR0132"  Part="1"
+AR Path="/5FFBF36C/5DAC5A6E" Ref="#PWR?"  Part="1"
+AR Path="/5DAC4399/5DAC5A6E" Ref="#PWR055"  Part="1"
+F 0 "#PWR0132" H 5250 2700 50  0001 C CNN
 F 1 "+3.3V" H 5265 3023 50  0000 C CNN
 F 2 "" H 5250 2850 50  0001 C CNN
@@
 P 4750 3450
 AR Path="/5DAC5A74" Ref="#PWR?"  Part="1"
-AR Path="/5DAA9390/5DAC4399/5DAC5A74" Ref="#PWR0148"  Part="1"
-F 0 "#PWR?" H 4750 3300 50  0001 C CNN
+AR Path="/5DAA9390/5DAC4399/5DAC5A74" Ref="#PWR0133"  Part="1"
+AR Path="/5FFBF36C/5DAC5A74" Ref="#PWR?"  Part="1"
+AR Path="/5DAC4399/5DAC5A74" Ref="#PWR053"  Part="1"
+F 0 "#PWR0133" H 4750 3300 50  0001 C CNN
 F 1 "+3.3V" H 4765 3623 50  0000 C CNN
 F 2 "" H 4750 3450 50  0001 C CNN
@@
 P 5950 3850
 AR Path="/5DAC5A7A" Ref="#PWR?"  Part="1"
-AR Path="/5DAA9390/5DAC4399/5DAC5A7A" Ref="#PWR0149"  Part="1"
-F 0 "#PWR?" H 5950 3600 50  0001 C CNN
+AR Path="/5DAA9390/5DAC4399/5DAC5A7A" Ref="#PWR0134"  Part="1"
+AR Path="/5FFBF36C/5DAC5A7A" Ref="#PWR?"  Part="1"
+AR Path="/5DAC4399/5DAC5A7A" Ref="#PWR059"  Part="1"
+F 0 "#PWR0134" H 5950 3600 50  0001 C CNN
 F 1 "GND" V 5950 3700 50  0000 R CNN
 F 2 "" H 5950 3850 50  0001 C CNN
@@
 P 5950 3950
 AR Path="/5DAC5A80" Ref="#PWR?"  Part="1"
-AR Path="/5DAA9390/5DAC4399/5DAC5A80" Ref="#PWR0150"  Part="1"
-F 0 "#PWR?" H 5950 3700 50  0001 C CNN
+AR Path="/5DAA9390/5DAC4399/5DAC5A80" Ref="#PWR0135"  Part="1"
+AR Path="/5FFBF36C/5DAC5A80" Ref="#PWR?"  Part="1"
+AR Path="/5DAC4399/5DAC5A80" Ref="#PWR060"  Part="1"
+F 0 "#PWR0135" H 5950 3700 50  0001 C CNN
 F 1 "GND" V 5955 3822 50  0000 R CNN
 F 2 "" H 5950 3950 50  0001 C CNN
@@
 P 6100 4050
 AR Path="/5DAC5A86" Ref="C?"  Part="1"
-AR Path="/5DAA9390/5DAC4399/5DAC5A86" Ref="C7"  Part="1"
-F 0 "C?" V 6250 3950 50  0000 C CNN
+AR Path="/5DAA9390/5DAC4399/5DAC5A86" Ref="C14"  Part="1"
+AR Path="/5FFBF36C/5DAC5A86" Ref="C?"  Part="1"
+AR Path="/5DAC4399/5DAC5A86" Ref="C14"  Part="1"
+F 0 "C14" V 6250 3950 50  0000 C CNN
 F 1 "0.1uF" V 6250 4050 50  0000 C CNN
 F 2 "Capacitor_SMD:C_0402_1005Metric" H 6138 3900 50  0001 C CNN
@@
 P 6250 4050
 AR Path="/5DAC5A8C" Ref="#PWR?"  Part="1"
-AR Path="/5DAA9390/5DAC4399/5DAC5A8C" Ref="#PWR0151"  Part="1"
-F 0 "#PWR?" H 6250 3800 50  0001 C CNN
+AR Path="/5DAA9390/5DAC4399/5DAC5A8C" Ref="#PWR0136"  Part="1"
+AR Path="/5FFBF36C/5DAC5A8C" Ref="#PWR?"  Part="1"
+AR Path="/5DAC4399/5DAC5A8C" Ref="#PWR061"  Part="1"
+F 0 "#PWR0136" H 6250 3800 50  0001 C CNN
 F 1 "GND" H 6255 3877 50  0000 C CNN
 F 2 "" H 6250 4050 50  0001 C CNN
@@
 P 5450 2850
 AR Path="/5DAC5A92" Ref="#PWR?"  Part="1"
-AR Path="/5DAA9390/5DAC4399/5DAC5A92" Ref="#PWR0152"  Part="1"
-F 0 "#PWR?" H 5450 2700 50  0001 C CNN
+AR Path="/5DAA9390/5DAC4399/5DAC5A92" Ref="#PWR0137"  Part="1"
+AR Path="/5FFBF36C/5DAC5A92" Ref="#PWR?"  Part="1"
+AR Path="/5DAC4399/5DAC5A92" Ref="#PWR057"  Part="1"
+F 0 "#PWR0137" H 5450 2700 50  0001 C CNN
 F 1 "+3.3V" H 5465 3023 50  0000 C CNN
 F 2 "" H 5450 2850 50  0001 C CNN

Commit message: rev ordered
Parts:
- U2: symbol SmallKat-v2-rescue:BNO055-Sensor_Motion-SmallKat-v2-rescue-SmallKat-v2-rescue-SmallKat-v2-rescue-SmallKat-v2-rescue-SmallKat-v2-rescue-SmallKat-v2-rescue-SmallKat-v2-rescue-SmallKat-v2-rescue -> SmallKat-v2-rescue:BNO055-Sensor_Motion-SmallKat-v2-rescue-SmallKat-v2-rescue-SmallKat-v2-rescue-SmallKat-v2-rescue-SmallKat-v2-rescue-SmallKat-v2-rescue-SmallKat-v2-rescue-SmallKat-v2-rescue-SmallKat-v2-rescue
Changed lines of the file:
@@
 $Descr A4 11693 8268
 encoding utf-8
-Sheet 3 7
+Sheet 4 7
 Title ""
 Date ""
@@
 $EndDescr
 $Comp
-L SmallKat-v2-rescue:BNO055-Sensor_Motion-SmallKat-v2-rescue-SmallKat-v2-rescue-SmallKat-v2-rescue-SmallKat-v2-rescue-SmallKat-v2-rescue-SmallKat-v2-rescue-SmallKat-v2-rescue-SmallKat-v2-rescue U?
+L SmallKat-v2-rescue:BNO055-Sensor_Motion-SmallKat-v2-rescue-SmallKat-v2-rescue-SmallKat-v2-rescue-SmallKat-v2-rescue-SmallKat-v2-rescue-SmallKat-v2-rescue-SmallKat-v2-rescue-SmallKat-v2-rescue-SmallKat-v2-rescue U?
 U 1 1 5DAC5A25
 P 5350 3550

Commit message: Final order version with all bom files
Parts:
- U2: symbol SmallKat-v2-rescue:BNO055-Sensor_Motion-SmallKat-v2-rescue-SmallKat-v2-rescue-SmallKat-v2-rescue-SmallKat-v2-rescue-SmallKat-v2-rescue-SmallKat-v2-rescue-SmallKat-v2-rescue-SmallKat-v2-rescue-SmallKat-v2-rescue -> SmallKat-v2-rescue:BNO055-Sensor_Motion-SmallKat-v2-rescue-SmallKat-v2-rescue-SmallKat-v2-rescue-SmallKat-v2-rescue-SmallKat-v2-rescue-SmallKat-v2-rescue-SmallKat-v2-rescue-SmallKat-v2-rescue-SmallKat-v2-rescue-SmallKat-v2-rescue-SmallKat-v2-rescue-SmallKat-v2-rescue-SmallKat-v2-rescue-SmallKat-v2-rescue
Changed lines of the file:
@@
 $EndDescr
 $Comp
-L SmallKat-v2-rescue:BNO055-Sensor_Motion-SmallKat-v2-rescue-SmallKat-v2-rescue-SmallKat-v2-rescue-SmallKat-v2-rescue-SmallKat-v2-rescue-SmallKat-v2-rescue-SmallKat-v2-rescue-SmallKat-v2-rescue-SmallKat-v2-rescue U?
+L SmallKat-v2-rescue:BNO055-Sensor_Motion-SmallKat-v2-rescue-SmallKat-v2-rescue-SmallKat-v2-rescue-SmallKat-v2-rescue-SmallKat-v2-rescue-SmallKat-v2-rescue-SmallKat-v2-rescue-SmallKat-v2-rescue-SmallKat-v2-rescue-SmallKat-v2-rescue-SmallKat-v2-rescue-SmallKat-v2-rescue-SmallKat-v2-rescue-SmallKat-v2-rescue U?
 U 1 1 5DAC5A25
 P 5350 3550
