File: MainBoard.kicad_sch (KiCad schematic)
At the start: 26 parts, among them J1 BATT_SERIAL, J25 Conn_01x02_Female, J3 Conn_01x03_Male, J4 Conn_01x03_Male, J5 Conn_01x03_Male, J6 Conn_01x03_Male

Commit message: Addressing the issues with the sample version, Updating the bom to source all the correct components from the JLCPCB supply
Parts:
- added J2: BATT_SERIAL, Connector_Molex:Molex_PicoBlade_53398-0271_1x02-1MP_P1.25mm_Vertical, symbol Connector:Conn_01x02_Female
- H1, H2, H3, H4, TP1, TP2, TP3: now left out of the parts list
- J1: footprint Connector_JST:JST_PH_B2B-PH-SM4-TB_1x02-1MP_P2.00mm_Vertical -> Connector_Molex:Molex_PicoBlade_53398-0271_1x02-1MP_P1.25mm_Vertical
- R3: value 2.4K -> 2.18K
Connections:
- net +BATT: now also J25.1 (Pin_1); no longer J25.2 (Pin_2)
- net BATT_SERIAL_RX: now also J1.1 (Pin_1); no longer J1.2 (Pin_2)
- net BATT_SERIAL_TX: now also J1.2 (Pin_2); no longer J1.1 (Pin_1)
- net GND: now also J25.2 (Pin_2), J2.2 (Pin_2); no longer J25.1 (Pin_1)
- new net +3V3: J2.1 (Pin_1)
- no-connect marks 0 -> 2
Other:
- sheet ESP32Module ports: added IO45, IO46; removed IO41, IO42
- note added: "Battery Communication"
- moved on the sheet: J25
Changed lines of the file:
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@@
   (junction (at 31.8516 76.1746) (diameter 0) (color 0 0 0 0)
   )
+  (no_connect (at 46.99 80.01))
+  (no_connect (at 46.99 81.915))
   (polyline (pts (xy 11.43 132.08) (xy 81.28 132.08))
     (stroke (width 0) (type default) (color 0 0 0 0))
@@
     (stroke (width 0) (type default) (color 0 0 0 0))
   )
+  (wire (pts (xy 154.3812 151.0284) (xy 154.3812 153.5684))
+    (stroke (width 0) (type default) (color 0 0 0 0))
+  )
   (wire (pts (xy 236.22 63.5) (xy 236.22 67.31))
     (stroke (width 0) (type default) (color 0 0 0 0))
@@
     (stroke (width 0) (type default) (color 0 0 0 0))
   )
+  (polyline (pts (xy 176.53 173.9392) (xy 176.53 142.1892))
+    (stroke (width 0) (type default) (color 0 0 0 0))
+  )
   (polyline (pts (xy 176.53 142.24) (xy 176.53 101.6))
     (stroke (width 0) (type default) (color 0 0 0 0))
@@
   )
   (polyline (pts (xy 135.89 199.39) (xy 179.07 199.39))
+    (stroke (width 0) (type default) (color 0 0 0 0))
+  )
+  (polyline (pts (xy 135.6868 173.9392) (xy 176.53 173.9392))
     (stroke (width 0) (type default) (color 0 0 0 0))
   )
@@
     (effects (font (size 2.9972 2.9972) (thickness 0.5994) bold) (justify left bottom))
   )
+  (text "    Battery\nCommunication" (at 138.0744 172.974 0)
+    (effects (font (size 2.9972 2.9972) (thickness 0.5994) bold) (justify left bottom))
+  )
   (text "Battery" (at 17.78 130.81 0)
     (effects (font (size 2.9972 2.9972) (thickness 0.5994) bold) (justify left bottom))
@@
     (effects (font (size 1.27 1.27)) (justify right bottom))
   )
-  (label "BATT_SERIAL_RX" (at 66.9544 113.1824 270)
-    (effects (font (size 1.27 1.27)) (justify right bottom))
-  )
-  (label "BATT_SERIAL_TX" (at 64.4144 113.1824 270)
+  (label "BATT_SERIAL_RX" (at 64.4144 113.1824 270)
+    (effects (font (size 1.27 1.27)) (justify right bottom))
+  )
+  (label "BATT_SERIAL_TX" (at 66.9544 113.1824 270)
     (effects (font (size 1.27 1.27)) (justify right bottom))
   )
@@
   )
   (symbol (lib_id "Connector:TestPoint") (at 250.19 85.09 0) (unit 1)
-    (in_bom yes) (on_board yes)
+    (in_bom no) (on_board yes)
     (property "Reference" "TP2" (id 0) (at 251.6632 82.0928 0)
       (effects (font (size 1.27 1.27)) (justify left))
@@
   )
   (symbol (lib_id "Connector:TestPoint") (at 259.08 85.09 0) (unit 1)
-    (in_bom yes) (on_board yes)
+    (in_bom no) (on_board yes)
     (property "Reference" "TP3" (id 0) (at 260.5532 82.0928 0)
       (effects (font (size 1.27 1.27)) (justify left))
@@
   )
   (symbol (lib_id "Mechanical:MountingHole_Pad") (at 55.88 139.7 0) (unit 1)
-    (in_bom yes) (on_board yes)
+    (in_bom no) (on_board yes)
     (property "Reference" "H3" (id 0) (at 58.42 138.4554 0)
       (effects (font (size 1.27 1.27)) (justify left))
@@
   )
   (symbol (lib_id "Mechanical:MountingHole_Pad") (at 30.48 139.7 0) (unit 1)
-    (in_bom yes) (on_board yes)
+    (in_bom no) (on_board yes)
     (property "Reference" "H1" (id 0) (at 33.02 138.4554 0)
       (effects (font (size 1.27 1.27)) (justify left))
@@
   )
   (symbol (lib_id "Mechanical:MountingHole_Pad") (at 55.88 153.67 0) (unit 1)
-    (in_bom yes) (on_board yes)
+    (in_bom no) (on_board yes)
     (property "Reference" "H4" (id 0) (at 58.42 152.4254 0)
       (effects (font (size 1.27 1.27)) (justify left))
@@
   )
   (symbol (lib_id "Mechanical:MountingHole_Pad") (at 30.48 153.67 0) (unit 1)
-    (in_bom yes) (on_board yes)
+    (in_bom no) (on_board yes)
     (property "Reference" "H2" (id 0) (at 33.02 152.4254 0)
       (effects (font (size 1.27 1.27)) (justify left))
@@
   )
   (symbol (lib_id "Connector:TestPoint") (at 31.8516 76.1746 180) (unit 1)
-    (in_bom yes) (on_board yes)
+    (in_bom no) (on_board yes)
     (property "Reference" "TP1" (id 0) (at 33.909 77.597 0))
     (property "Value" "Check for life" (id 1) (at 24.257 79.375 0))
@@
       (effects (font (size 1.27 1.27)) (justify left))
     )
-    (property "Value" "2.4K" (id 1) (at 89.408 161.163 0)
+    (property "Value" "2.18K" (id 1) (at 89.408 161.163 0)
       (effects (font (size 1.27 1.27)) (justify left))
     )
@@
     (pin "3")
   )
-  (symbol (lib_id "Connector:Conn_01x02_Female") (at 29.21 107.95 270) (mirror x) (unit 1)
-    (in_bom yes) (on_board yes)
-    (property "Reference" "J25" (id 0) (at 26.67 102.87 90)
-      (effects (font (size 1.27 1.27)) (justify left))
-    )
-    (property "Value" "Conn_01x02_Female" (id 1) (at 19.05 105.41 90)
-      (effects (font (size 1.27 1.27)) (justify left))
-    )
-    (property "Footprint" "RC-Battery-Connectors:XT-60_male" (id 2) (at 29.21 107.95 0)
-      (effects (font (size 1.27 1.27)) hide)
-    )
-    (property "Datasheet" "~" (id 3) (at 29.21 107.95 0)
+  (symbol (lib_id "Connector:Conn_01x02_Female") (at 26.67 107.95 90) (unit 1)
+    (in_bom yes) (on_board yes)
+    (property "Reference" "J25" (id 0) (at 29.21 102.87 90)
+      (effects (font (size 1.27 1.27)) (justify left))
+    )
+    (property "Value" "Conn_01x02_Female" (id 1) (at 36.83 105.41 90)
+      (effects (font (size 1.27 1.27)) (justify left))
+    )
+    (property "Footprint" "RC-Battery-Connectors:XT-60_male" (id 2) (at 26.67 107.95 0)
+      (effects (font (size 1.27 1.27)) hide)
+    )
+    (property "Datasheet" "~" (id 3) (at 26.67 107.95 0)
       (effects (font (size 1.27 1.27)) hide)
     )
@@
     (pin "2")
   )
+  (symbol (lib_id "power:+3V3") (at 154.3812 153.5684 180) (unit 1)
+    (in_bom yes) (on_board yes) (fields_autoplaced)
+    (property "Reference" "#PWR0157" (id 0) (at 154.3812 149.7584 0)
+      (effects (font (size 1.27 1.27)) hide)
+    )
+    (property "Value" "+3V3" (id 1) (at 154.3812 158.5468 0))
+    (property "Footprint" "" (id 2) (at 154.3812 153.5684 0)
+      (effects (font (size 1.27 1.27)) hide)
+    )
+    (property "Datasheet" "" (id 3) (at 154.3812 153.5684 0)
+      (effects (font (size 1.27 1.27)) hide)
+    )
+    (pin "1")
+  )
+  (symbol (lib_id "Connector:Conn_01x02_Female") (at 154.3812 145.9484 90) (unit 1)
+    (in_bom yes) (on_board yes)
+    (property "Reference" "J2" (id 0) (at 158.496 149.2504 90)
+      (effects (font (size 1.27 1.27)) (justify right))
+    )
+    (property "Value" "BATT_SERIAL" (id 1) (at 150.114 144.5768 90)
+      (effects (font (size 1.27 1.27)) (justify right))
+    )
+    (property "Footprint" "Connector_Molex:Molex_PicoBlade_53398-0271_1x02-1MP_P1.25mm_Vertical" (id 2) (at 154.3812 145.9484 0)
+      (effects (font (size 1.27 1.27)) hide)
+    )
+    (property "Datasheet" "~" (id 3) (at 154.3812 145.9484 0)
+      (effects (font (size 1.27 1.27)) hide)
+    )
+    (pin "1")
+    (pin "2")
+  )
   (symbol (lib_id "Connector:Conn_01x02_Female") (at 64.4144 108.1024 90) (unit 1)
     (in_bom yes) (on_board yes)
@@
       (effects (font (size 1.27 1.27)) (justify right))
     )
-    (property "Footprint" "Connector_JST:JST_PH_B2B-PH-SM4-TB_1x02-1MP_P2.00mm_Vertical" (id 2) (at 64.4144 108.1024 0)
+    (property "Footprint" "Connector_Molex:Molex_PicoBlade_53398-0271_1x02-1MP_P1.25mm_Vertical" (id 2) (at 64.4144 108.1024 0)
       (effects (font (size 1.27 1.27)) hide)
     )
@@
     (pin "1")
     (pin "2")
+  )
+  (symbol (lib_id "power:GND") (at 156.9212 151.0284 0) (unit 1)
+    (in_bom yes) (on_board yes) (fields_autoplaced)
+    (property "Reference" "#PWR0158" (id 0) (at 156.9212 157.3784 0)
+      (effects (font (size 1.27 1.27)) hide)
+    )
+    (property "Value" "GND" (id 1) (at 156.9212 156.0068 0))
+    (property "Footprint" "" (id 2) (at 156.9212 151.0284 0)
+      (effects (font (size 1.27 1.27)) hide)
+    )
+    (property "Datasheet" "" (id 3) (at 156.9212 151.0284 0)
+      (effects (font (size 1.27 1.27)) hide)
+    )
+    (pin "1")
   )
   (sheet (at 46.99 20.32) (size 40.64 70.485) (fields_autoplaced)
@@
       (effects (font (size 1.27 1.27)) (justify left))
     )
-    (pin "IO41" input (at 46.99 80.01 180)
-      (effects (font (size 1.27 1.27)) (justify left))
-    )
-    (pin "IO42" input (at 46.99 81.915 180)
-      (effects (font (size 1.27 1.27)) (justify left))
-    )
     (pin "IO47" input (at 46.99 83.82 180)
       (effects (font (size 1.27 1.27)) (justify left))
@@
       (effects (font (size 1.27 1.27)) (justify left))
     )
+    (pin "IO45" input (at 46.99 80.01 180)
+      (effects (font (size 1.27 1.27)) (justify left))
+    )
+    (pin "IO46" input (at 46.99 81.915 180)
+      (effects (font (size 1.27 1.27)) (justify left))
+    )

Commit message: Adding usb c pd negotiation for battery charging
Parts:
- F1: footprint 01550900M:0154.250DR -> 0155.500:0154500DRTL
- J25: footprint RC-Battery-Connectors:XT-60_male -> Connector_AMASS:AMASS_XT30U-F_1x02_P5.0mm_Vertical
Connections:
- net ESP32Module/IO36 is gone; now on net ESP32Module/IO45: R1.1, TP1.1
- net +BATT: now also J25.2 (Pin_2); no longer J25.1 (Pin_1)
- net GND: now also J25.1 (Pin_1); no longer J25.2 (Pin_2)
Other:
- sheet sheet5E0C1128 renamed 6V Switchmode
- added sheet USB_PD (USB_PD.kicad_sch)
- sheet ESP32Module ports: added USBD_N, USBD_P; removed none
- moved on the sheet: D1, J25, R1, TP1
