File: Servos.kicad_sch (KiCad schematic)
At the start: 36 parts, among them J10 Conn_01x03_Male, J11 Conn_01x03_Male, J12 Conn_01x03_Male, J13 Conn_01x03_Male, J14 Conn_01x03_Male, J15 Conn_01x03_Male, J16 Conn_01x03_Male, J17 Conn_01x03_Male, J18 Conn_01x03_Male, J19 Conn_01x03_Male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

Commit message: Adding usb c pd negotiation for battery charging
Parts:
- F2, F3, F4, F5: footprint 01550900M:0154.250DR -> 0155.500:0154500DRTL
